Commit message: update to support latest iDynTree and load update model for iCubGenova03

File: app/robots/iCubGenova03/model.urdf (robot description, URDF)
Before this commit: robot test_icub, 46 links, 45 joints
Links:
- link l_foot: mass -0.09 -> 0.761
- link r_foot: mass -0.09 -> 0.761
- link root_link: mass 1.2 -> 4.72
Joints:
- joint l_foot_ft_sensor: origin xyz=0 0 0.041 rpy=0 1.5708 0 -> xyz=-0.0035 0 0.0685 rpy=0 1.5708 0
- joint r_foot_ft_sensor: origin xyz=0 0 0.041 rpy=0 1.5708 0 -> xyz=-0.0035 4.28626e-19 0.0685 rpy=0 1.5708 0
