Commit message: [iCubHeidelberg01] updated model

File: app/robots/iCubHeidelberg01/model.urdf (robot description, URDF)
Before this commit: robot iCubHeidelberg01_SIM_MODEL, 73 links, 72 joints
Links:
- removed link SCSYS_EMS_ACCEL
- removed link SCSYS_EMS_ACCEL0
- removed link SCSYS_EMS_ACCEL1
- removed link SCSYS_EMS_ACCEL2
- removed link SCSYS_EMS_ACCEL3
- removed link SCSYS_EMS_ACCEL_1
- removed link SCSYS_EMS_ACCEL_10
- removed link SCSYS_EMS_ACCEL_11
- removed link SCSYS_EMS_GYRO
- removed link SCSYS_EMS_GYRO0
- removed link SCSYS_EMS_GYRO1
- removed link SCSYS_EMS_GYRO2
- removed link SCSYS_EMS_GYRO3
- removed link SCSYS_EMS_GYRO_1
- removed link SCSYS_EMS_GYRO_10
- removed link SCSYS_EMS_GYRO_11
- removed link SCSYS_MTB_ACCEL
- removed link SCSYS_MTB_ACCEL0
- removed link SCSYS_MTB_ACCEL1
- removed link SCSYS_MTB_ACCEL2
- removed link SCSYS_MTB_ACCEL3
- removed link SCSYS_MTB_ACCEL4
- removed link SCSYS_MTB_ACCEL_1
- removed link SCSYS_MTB_ACCEL_10
- removed link SCSYS_MTB_ACCEL_11
- removed link SCSYS_MTB_ACCEL_12
- removed link SCSYS_MTB_ACCEL_13
- removed link SCSYS_MTB_ACCEL_14
- removed link SCSYS_MTB_ACCEL_2
- removed link SCSYS_MTB_ACCEL_20
- removed link SCSYS_MTB_ACCEL_21
- removed link SCSYS_MTB_ACCEL_22
- removed link SCSYS_MTB_ACCEL_3
- removed link SCSYS_MTB_ACCEL_30
- removed link SCSYS_MTB_ACCEL_31
- removed link SCSYS_MTB_ACCEL_32
- removed link SCSYS_MTB_ACCEL_4
- removed link SCSYS_MTB_ACCEL_40
- removed link SCSYS_MTB_ACCEL_5
- removed link SCSYS_MTB_ACCEL_50
- removed link SCSYS_MTB_ACCEL_6
- removed link SCSYS_MTB_ACCEL_60
- removed link SCSYS_MTB_ACCEL_7
- removed link SCSYS_MTB_ACCEL_70
- removed link SCSYS_MTX_ACCEL_0
- removed link base_link
- removed link l_ankle
- removed link l_shank
- removed link l_thigh
- removed link l_upper_foot
- removed link l_upper_thigh
- removed link lap_belt_1
- removed link lap_belt_2
- removed link r_ankle
- removed link r_shank
- removed link r_thigh
- removed link r_upper_foot
- removed link r_upper_thigh
- added link l_ankle_1, mass 0.8929; collision mesh filename=model://iCubHeidelberg01_model/dae_meshes/sim_sea_l_ankle_p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 scale=0.001 0.001 0.001; visual mesh filename=model://iCubHeidelberg01_model/dae_meshes/sim_sea_l_ankle_p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 scale=0.001 0.001 0.001
- added link l_ankle_2, mass 0.2675; collision mesh filename=model://iCubHeidelberg01_model/dae_meshes/sim_sea_l_foot_pr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 scale=0.001 0.001 0.001; visual mesh filename=model://iCubHeidelberg01_model/dae_meshes/sim_sea_l_foot_pr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 scale=0.001 0.001 0.001
- added link l_hip_3, mass 0.1262; collision mesh filename=model://iCubHeidelberg01_model/dae_meshes/sim_sea_l_upper_t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 scale=0.001 0.001 0.001; visual mesh filename=model://iCubHeidelberg01_model/dae_meshes/sim_sea_l_upper_t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 scale=0.001 0.001 0.001
- added link l_lower_leg, mass 1.7086; collision mesh filename=model://iCubHeidelberg01_model/dae_meshes/sim_sea_l_shank_p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 scale=0.001 0.001 0.001; visual mesh filename=model://iCubHeidelberg01_model/dae_meshes/sim_sea_l_shank_p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 scale=0.001 0.001 0.001
- added link l_sole
- added link l_upper_leg, mass 2.2544; collision mesh filename=model://iCubHeidelberg01_model/dae_meshes/sim_sea_l_thigh_p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 scale=0.001 0.001 0.001; visual mesh filename=model://iCubHeidelberg01_model/dae_meshes/sim_sea_l_thigh_p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 scale=0.001 0.001 0.001
- added link r_ankle_1, mass 0.8929; collision mesh filename=model://iCubHeidelberg01_model/dae_meshes/sim_sea_r_ankle_p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 scale=0.001 0.001 0.001; visual mesh filename=model://iCubHeidelberg01_model/dae_meshes/sim_sea_r_ankle_p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 scale=0.001 0.001 0.001
- added link r_ankle_2, mass 0.2675; collision mesh filename=model://iCubHeidelberg01_model/dae_meshes/sim_sea_r_foot_pr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 scale=0.001 0.001 0.001; visual mesh filename=model://iCubHeidelberg01_model/dae_meshes/sim_sea_r_foot_pr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 scale=0.001 0.001 0.001
- added link r_hip_3, mass 0.1262; collision mesh filename=model://iCubHeidelberg01_model/dae_meshes/sim_sea_r_upper_t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 scale=0.001 0.001 0.001; visual mesh filename=model://iCubHeidelberg01_model/dae_meshes/sim_sea_r_upper_t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 scale=0.001 0.001 0.001
- added link r_lower_leg, mass 1.7086; collision mesh filename=model://iCubHeidelberg01_model/dae_meshes/sim_sea_r_shank_p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 scale=0.001 0.001 0.001; visual mesh filename=model://iCubHeidelberg01_model/dae_meshes/sim_sea_r_shank_p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 scale=0.001 0.001 0.001
- added link r_sole
- added link r_upper_leg, mass 2.2544; collision mesh filename=model://iCubHeidelberg01_model/dae_meshes/sim_sea_r_thigh_p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 scale=0.001 0.001 0.001; visual mesh filename=model://iCubHeidelberg01_model/dae_meshes/sim_sea_r_thigh_p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 scale=0.001 0.001 0.001
- added link torso_1, mass 0.7112; collision mesh filename=model://iCubHeidelberg01_model/dae_meshes/sim_lap_belt_1_pr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 scale=0.001 0.001 0.001; visual mesh filename=model://iCubHeidelberg01_model/dae_meshes/sim_lap_belt_1_pr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 scale=0.001 0.001 0.001
- added link torso_2, mass 0.3954; collision mesh filename=model://iCubHeidelberg01_model/dae_meshes/sim_lap_belt_2_pr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 scale=0.001 0.001 0.001; visual mesh filename=model://iCubHeidelberg01_model/dae_meshes/sim_lap_belt_2_pr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 scale=0.001 0.001 0.001
- link chest: mass 9.71648 -> 6.1306; geometry collision mesh filename=model://iCubHeidelberg01_model/dae_meshes/sim_chest__prt.dae scale=0.001 0.001 0.001; visual mesh filename=model://iCubHeidelberg01_model/dae_meshes/sim_chest__prt.dae scale=0.001 0.001 0.001
- link l_foot: mass 0.907917 -> 0.3794
- link l_hip_1: mass 0.610394 -> 0.9279
- link l_hip_2: mass 0.292811 -> 0.4184
- link r_foot: mass 0.907917 -> 0.3794
- link r_hip_1: mass 0.610394 -> 0.9279
- link r_hip_2: mass 0.292811 -> 0.4184
- link root_link: mass 4.55132 -> 5.1504; geometry collision mesh filename=model://iCubHeidelberg01_model/dae_meshes/sim_root_link_prt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 scale=0.001 0.001 0.001; visual mesh filename=model://iCubHeidelberg01_model/dae_meshes/sim_root_link_prt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 scale=0.001 0.001 0.001
Joints:
- removed joint SCSYS_EMS_ACCEL0_fixed_joint
- removed joint SCSYS_EMS_ACCEL1_fixed_joint
- removed joint SCSYS_EMS_ACCEL2_fixed_joint
- removed joint SCSYS_EMS_ACCEL3_fixed_joint
- removed joint SCSYS_EMS_ACCEL_10_fixed_joint
- removed joint SCSYS_EMS_ACCEL_11_fixed_joint
- removed joint SCSYS_EMS_ACCEL_1_fixed_joint
- removed joint SCSYS_EMS_ACCEL_fixed_joint
- removed joint SCSYS_EMS_GYRO0_fixed_joint
- removed joint SCSYS_EMS_GYRO1_fixed_joint
- removed joint SCSYS_EMS_GYRO2_fixed_joint
- removed joint SCSYS_EMS_GYRO3_fixed_joint
- removed joint SCSYS_EMS_GYRO_10_fixed_joint
- removed joint SCSYS_EMS_GYRO_11_fixed_joint
- removed joint SCSYS_EMS_GYRO_1_fixed_joint
- removed joint SCSYS_EMS_GYRO_fixed_joint
- removed joint SCSYS_MTB_ACCEL0_fixed_joint
- removed joint SCSYS_MTB_ACCEL1_fixed_joint
- removed joint SCSYS_MTB_ACCEL2_fixed_joint
- removed joint SCSYS_MTB_ACCEL3_fixed_joint
- removed joint SCSYS_MTB_ACCEL4_fixed_joint
- removed joint SCSYS_MTB_ACCEL_10_fixed_joint
- removed joint SCSYS_MTB_ACCEL_11_fixed_joint
- removed joint SCSYS_MTB_ACCEL_12_fixed_joint
- removed joint SCSYS_MTB_ACCEL_13_fixed_joint
- removed joint SCSYS_MTB_ACCEL_14_fixed_joint
- removed joint SCSYS_MTB_ACCEL_1_fixed_joint
- removed joint SCSYS_MTB_ACCEL_20_fixed_joint
- removed joint SCSYS_MTB_ACCEL_21_fixed_joint
- removed joint SCSYS_MTB_ACCEL_22_fixed_joint
- removed joint SCSYS_MTB_ACCEL_2_fixed_joint
- removed joint SCSYS_MTB_ACCEL_30_fixed_joint
- removed joint SCSYS_MTB_ACCEL_31_fixed_joint
- removed joint SCSYS_MTB_ACCEL_32_fixed_joint
- removed joint SCSYS_MTB_ACCEL_3_fixed_joint
- removed joint SCSYS_MTB_ACCEL_40_fixed_joint
- removed joint SCSYS_MTB_ACCEL_4_fixed_joint
- removed joint SCSYS_MTB_ACCEL_50_fixed_joint
- removed joint SCSYS_MTB_ACCEL_5_fixed_joint
- removed joint SCSYS_MTB_ACCEL_60_fixed_joint
- removed joint SCSYS_MTB_ACCEL_6_fixed_joint
- removed joint SCSYS_MTB_ACCEL_70_fixed_joint
- removed joint SCSYS_MTB_ACCEL_7_fixed_joint
- removed joint SCSYS_MTB_ACCEL_fixed_joint
- removed joint SCSYS_MTX_ACCEL_0_fixed_joint
- removed joint base_fixed_joint
- added joint l_sole_fixed_joint: type fixed, parent l_foot, child l_sole, origin xyz=9.72e-05 0 0.014399 rpy=-3.14159265359 0.00674386312028 0
- added joint r_sole_fixed_joint: type fixed, parent r_foot, child r_sole, origin xyz=0 0 0.0144000000055 rpy=-3.14159265359 0 0
- joint l_ankle_pitch: axis -1.0 0.0 0.0 -> 1.0 0.0 0.0; child l_ankle -> l_ankle_1; origin xyz=-0.0129305 -0.2005 0 rpy=0 0 0 -> xyz=-0.021343 -0.200983719847 0.00294927094483 rpy=2.4080004131e-05 0 0; parent l_shank -> l_lower_leg
- joint l_ankle_roll: axis -0.0 1.23785e-12 -1.0 -> -0.0 0 -1; child l_upper_foot -> l_ankle_2; origin xyz=0.02702 0 -0.044562467 rpy=0 0 0 -> xyz=0.0355 -1.6398477099e-05 -0.0475117797388 rpy=0 0 0; parent l_ankle -> l_ankle_1
- joint l_foot_ft_sensor: origin xyz=0.0701 0.587138 0.000853467382024 rpy=0 0 0 -> xyz=0 -0.0603002589183 0.0480625407102 rpy=0 1.5640527248 -1.57079632679; parent l_upper_foot -> l_ankle_2
- joint l_hip_pitch: origin xyz=-0.026 -0.151913 -0.0428515 rpy=3.14159265359 0 3.14159265359 -> xyz=0.0064515 -0.0111 -0.119913 rpy=1.57751584879 0 1.57079632679
- joint l_hip_roll: axis -0.0 1.26404e-12 -1.0 -> -0.0 0 -1; origin xyz=-0.0961 0 0.0262471 rpy=0 0 0 -> xyz=-0.059 -8.59963575406e-07 0.026362200929 rpy=0 0 0
- joint l_hip_yaw: axis -0.0 1.0 1.22451e-12 -> -0.0 1 0; child l_thigh -> l_upper_leg; origin xyz=-0.0701 -0.244213 0.0437089998092 rpy=0 0 0 -> xyz=0.000121 0 0.017999 rpy=-1.5640768048 0 1.57079632679; parent l_upper_thigh -> l_hip_3
- joint l_knee: child l_shank -> l_lower_leg; origin xyz=-0.0178895 -0.145625 0 rpy=0 0 0 -> xyz=-0.017957 -0.145625287455 0 rpy=0 0 0; parent l_thigh -> l_upper_leg
- joint l_leg_ft_sensor: child l_upper_thigh -> l_hip_3; origin xyz=0.0701 0.151913 -0.0690985998093 rpy=0 0 0 -> xyz=0 -0.0743000549473 -0.0255046186937 rpy=0 1.5640768048 -1.57079632679
- joint r_ankle_pitch: child r_ankle -> r_ankle_1; origin xyz=-0.0129305 -0.2005 0 rpy=0 0 0 -> xyz=-0.021343 -0.201 0 rpy=-2.40788999988e-05 0 0; parent r_shank -> r_lower_leg
- joint r_ankle_roll: axis -0.0 -0.0 -1.0 -> 0.0 0 -1.0; child r_upper_foot -> r_ankle_2; origin xyz=0.02702 0 0.044562467 rpy=0 0 0 -> xyz=0.0355 0 0.0445624670112 rpy=0 0 0; parent r_ankle -> r_ankle_1
- joint r_foot_ft_sensor: origin xyz=0.0701 0.587138 -0.000853467381377 rpy=0 0 0 -> xyz=0 -0.0603008427249 -0.0480625189919 rpy=3.14159265359 -1.57079632651 -1.57079632679; parent r_upper_foot -> r_ankle_2
- joint r_hip_pitch: axis -1.0 -0.0 -0.0 -> 1.0 0.0 0.0; origin xyz=-0.0262461 -0.151913 -0.0428515 rpy=0 0 0 -> xyz=0.0064515 0.0111 -0.119913 rpy=1.57079632679 0 -1.57079632679
- joint r_hip_roll: axis 0.0 0.0 -1.0 -> 0.0 0.0 1.0; origin xyz=-0.0438539 0 -0.0262471 rpy=0 0 0 -> xyz=-0.059 0 -0.0263622 rpy=0 0 0
- joint r_hip_yaw: child r_thigh -> r_upper_leg; origin xyz=-0.0701 -0.244213 -0.0437089998094 rpy=0 0 0 -> xyz=0 0 0.018 rpy=-1.57079632679 0 -1.57079632679; parent r_upper_thigh -> r_hip_3
- joint r_knee: child r_shank -> r_lower_leg; origin xyz=-0.0178895 -0.145625 0 rpy=0 0 0 -> xyz=-0.017957 -0.145625 0 rpy=0 0 0; parent r_thigh -> r_upper_leg
- joint r_leg_ft_sensor: child r_upper_thigh -> r_hip_3; origin xyz=0.0701 0.151913 0.0690985998094 rpy=0 0 0 -> xyz=0 -0.0743 0.0255047 rpy=1.57079632679 -1.57079632679 0
- joint torso_pitch: child lap_belt_1 -> torso_1; origin xyz=-0.0394 -0.032 -0.0364 rpy=0 0 0 -> xyz=0 0.0394 0 rpy=1.57079632663 0 -1.57079632679
- joint torso_roll: axis 0.0 -1.61681e-10 -1.0 -> 0.0 0 -1.0; child lap_belt_2 -> torso_2; origin xyz=0.0393999998093 0.032 -0.0538389999948 rpy=0 0 0 -> xyz=0.0393999998093 0.032 -0.0587918999948 rpy=0 0 0; parent lap_belt_1 -> torso_1
- joint torso_yaw: axis 0.0 -1.0 1.61681e-10 -> 0.0 -1.0 0; origin xyz=0 0.0519999999991 0.0593390000084 rpy=0 0 0 -> xyz=0 0.0514999999991 0.0642919000083 rpy=0 0 0; parent lap_belt_2 -> torso_2

Commit message: [iCubHeidelberg01] added base_link dummy link

File: app/robots/iCubHeidelberg01/model.urdf (robot description, URDF)
Before this commit: robot iCubHeidelberg01_SIM_MODEL, 29 links, 28 joints
Links:
- added link base_link
Joints:
- added joint base_fixed_joint: type fixed, parent base_link, child root_link, origin xyz=0 0 0 rpy=0 -0 0, axis 0 0 0

Commit message: [iCubHeidelberg01] added feet dh frames

File: app/robots/iCubHeidelberg01/model.urdf (robot description, URDF)
Before this commit: robot iCubHeidelberg01_SIM_MODEL, 30 links, 29 joints
Links:
- added link l_foot_dh_frame
- added link r_foot_dh_frame
Joints:
- added joint l_foot_dh_frame_fixed_joint: type fixed, parent l_foot, child l_foot_dh_frame, origin xyz=9.72e-05 0 0.014399 rpy=0.0 1.5708 0.0
- added joint r_foot_dh_frame_fixed_joint: type fixed, parent r_foot, child r_foot_dh_frame, origin xyz=0 0 0.0144000000055 rpy=0.0 1.5708 0.0

Commit message: [iCubHeidelberg01] commented out optional weights

File: app/robots/iCubHeidelberg01/model.urdf (robot description, URDF)
Before this commit: robot iCubHeidelberg01_SIM_MODEL, 32 links, 31 joints
Links:
- removed link WEIGHT-1KG
- removed link WEIGHT-1KG-1
- removed link WEIGHT-1KG-2
- removed link WEIGHT-1KG-3
- removed link WEIGHT-1KG-4
- removed link WEIGHT-1KG-5
Joints:
- removed joint chest_weight_1
- removed joint chest_weight_2
- removed joint chest_weight_3
- removed joint chest_weight_4
- removed joint chest_weight_5
- removed joint chest_weight_6

Commit message: [iCubHeidelberg01] fix wrong joint axis directions

File: app/robots/iCubHeidelberg01/model.urdf (robot description, URDF)
Before this commit: robot iCubHeidelberg01_SIM_MODEL, 26 links, 25 joints
Joints:
- joint l_ankle_pitch: axis 1.0 0.0 0.0 -> -1.0 0.0 0.0
- joint r_hip_pitch: axis 1.0 0.0 0.0 -> -1.0 0.0 0.0
- joint r_hip_roll: axis 0.0 0.0 1.0 -> 0.0 0.0 -1.0
