Commit message: Added urdf model for iCubParis01

File: app/robots/iCubParis01/model.urdf (robot description, URDF)
Before this commit: robot test_icub, 55 links, 54 joints
Links:
- link l_ankle_1: mass 0.643 -> 0.746
- link l_hip_1: mass 0.695 -> 0.754
- link l_hip_2: mass 0.982 -> 0.526
- link l_lower_leg: mass 2.032 -> 1.264
- link l_upper_leg: mass 1.522 -> 2.175
- link r_ankle_1: mass 0.643 -> 0.746
- link r_hip_1: mass 0.695 -> 0.754
- link r_hip_2: mass 0.982 -> 0.526
- link r_lower_leg: mass 2.032 -> 1.264
- link r_upper_leg: mass 1.522 -> 2.175
Joints:
- joint codyco_balancing_world_fixed_joint: origin xyz=-8.67362e-19 -1.38778e-17 0.075 rpy=3.14159 -0 0 -> xyz=-1.84889e-33 -1.38778e-17 0.075 rpy=3.14159 -0 0
- joint l_ankle_pitch: origin xyz=-0.2005 0 0 rpy=-1.5708 0 0 -> xyz=-0.213 0 0 rpy=-1.5708 0 0
- joint l_foot_dh_frame_fixed_joint: origin xyz=-8.67362e-19 -1.38778e-17 0.075 rpy=-9.70754e-18 1.5708 -9.70754e-18 -> xyz=-1.84889e-33 -1.38778e-17 0.075 rpy=-9.70754e-18 1.5708 -9.70754e-18
- joint l_hip_yaw: origin xyz=0 -1.68519e-34 -0.0665 rpy=-1.5708 -6.16298e-33 -6.12323e-17 -> xyz=0 0 -0.0665 rpy=-1.5708 -6.16298e-33 -6.12323e-17
- joint l_knee: origin xyz=-0.0009175 -0.234545 -1.43617e-17 rpy=3.14159 -1.2326e-32 1.5708 -> xyz=0 -0.2236 -1.36916e-17 rpy=3.14159 -1.2326e-32 1.5708
- joint r_ankle_pitch: origin xyz=-0.2005 0 0 rpy=1.5708 -0 0 -> xyz=-0.213 0 0 rpy=1.5708 -0 0
- joint r_foot_dh_frame_fixed_joint: origin xyz=-4.29004e-17 -0.1362 0.075 rpy=-0.834365 1.5708 -0.834365 -> xyz=-4.2033e-17 -0.1362 0.075 rpy=-0.834365 1.5708 -0.834365
- joint r_hip_yaw: origin xyz=0 1.68519e-34 -0.0665 rpy=-1.5708 -6.16298e-33 6.12323e-17 -> xyz=0 0 -0.0665 rpy=-1.5708 -6.16298e-33 6.12323e-17
- joint r_knee: origin xyz=-0.0009175 -0.234545 1.43617e-17 rpy=3.14159 -1.2326e-32 1.5708 -> xyz=0 -0.2236 1.36916e-17 rpy=3.14159 -1.2326e-32 1.5708

Commit message: update iCubParis* models after https://github.com/robotology-playground/icub-model-generator

File: app/robots/iCubParis01/model.urdf (robot description, URDF)
Before this commit: robot test_icub, 55 links, 54 joints
Links:
- link l_ankle_2: mass 0.1 -> 0.2675
- link l_foot: mass 0.761 -> 0.5935
- link r_ankle_2: mass 0.1 -> 0.2675
- link r_foot: mass 0.761 -> 0.5935
Joints:
- joint codyco_balancing_world_fixed_joint: origin xyz=-1.84889e-33 -1.38778e-17 0.075 rpy=3.14159 -0 0 -> xyz=-0.0353 -1.38778e-17 -0.001 rpy=3.14159 -0 0
- joint l_foot_dh_frame_fixed_joint: origin xyz=-1.84889e-33 -1.38778e-17 0.075 rpy=-9.70754e-18 1.5708 -9.70754e-18 -> xyz=-0.0353 0 -0.001 rpy=0 1.5708 0
- joint l_foot_ft_sensor: origin xyz=-0.0035 0 -0.0065 rpy=0 -0 0 -> xyz=0.0135 0 0.0695 rpy=0 -0 0
- joint l_sole_fixed_joint: origin xyz=0 0 0.075 rpy=0 1.5708 0 -> xyz=-0.0353 -1.38778e-17 -0.001 rpy=3.14159 -0 0
- joint r_foot_dh_frame_fixed_joint: origin xyz=-8.67362e-19 1.38778e-17 0.075 rpy=-1.01315e-16 1.5708 -1.01315e-16 -> xyz=-0.0353 0 -0.001 rpy=0 1.5708 0
- joint r_foot_ft_sensor: origin xyz=-0.0035 4.28626e-19 -0.0065 rpy=0 -0 0 -> xyz=0.0135 4.28626e-19 0.0695 rpy=0 -0 0
- joint r_sole_fixed_joint: origin xyz=0 0 0.075 rpy=0 1.5708 0 -> xyz=-0.0353 -1.38778e-17 -0.001 rpy=3.14159 -0 0

File: app/robots/iCubParis02/model.urdf (robot description, URDF)
Before this commit: robot test_icub, 55 links, 54 joints
Links:
- link l_ankle_1: mass 0.643 -> 0.746
- link l_ankle_2: mass 0.1 -> 0.2675
- link l_foot: mass 0.761 -> 0.5935
- link l_hip_1: mass 0.695 -> 0.754
- link l_hip_2: mass 0.982 -> 0.526
- link l_lower_leg: mass 2.032 -> 1.264
- link l_upper_leg: mass 1.522 -> 2.175
- link r_ankle_1: mass 0.643 -> 0.746
- link r_ankle_2: mass 0.1 -> 0.2675
- link r_foot: mass 0.761 -> 0.5935
- link r_hip_1: mass 0.695 -> 0.754
- link r_hip_2: mass 0.982 -> 0.526
- link r_lower_leg: mass 2.032 -> 1.264
- link r_upper_leg: mass 1.522 -> 2.175
Joints:
- joint codyco_balancing_world_fixed_joint: origin xyz=-8.67362e-19 -1.38778e-17 0.075 rpy=3.14159 -0 0 -> xyz=-0.0353 -1.38778e-17 -0.001 rpy=3.14159 -0 0
- joint l_ankle_pitch: origin xyz=-0.2005 0 0 rpy=-1.5708 0 0 -> xyz=-0.213 0 0 rpy=-1.5708 0 0
- joint l_foot_dh_frame_fixed_joint: origin xyz=-8.67362e-19 -1.38778e-17 0.075 rpy=-9.70754e-18 1.5708 -9.70754e-18 -> xyz=-0.0353 0 -0.001 rpy=0 1.5708 0
- joint l_foot_ft_sensor: origin xyz=-0.0035 0 -0.0065 rpy=0 -0 0 -> xyz=0.0135 0 0.0695 rpy=0 -0 0
- joint l_hip_yaw: origin xyz=0 -1.68519e-34 -0.0665 rpy=-1.5708 -6.16298e-33 -6.12323e-17 -> xyz=0 0 -0.0665 rpy=-1.5708 -6.16298e-33 -6.12323e-17
- joint l_knee: origin xyz=-0.0009175 -0.234545 -1.43617e-17 rpy=3.14159 -1.2326e-32 1.5708 -> xyz=0 -0.2236 -1.36916e-17 rpy=3.14159 -1.2326e-32 1.5708
- joint l_sole_fixed_joint: origin xyz=0 0 0.075 rpy=0 1.5708 0 -> xyz=-0.0353 -1.38778e-17 -0.001 rpy=3.14159 -0 0
- joint r_ankle_pitch: origin xyz=-0.2005 0 0 rpy=1.5708 -0 0 -> xyz=-0.213 0 0 rpy=1.5708 -0 0
- joint r_foot_dh_frame_fixed_joint: origin xyz=-8.67362e-19 1.38778e-17 0.075 rpy=-1.01315e-16 1.5708 -1.01315e-16 -> xyz=-0.0353 0 -0.001 rpy=0 1.5708 0
- joint r_foot_ft_sensor: origin xyz=-0.0035 4.28626e-19 -0.0065 rpy=0 -0 0 -> xyz=0.0135 4.28626e-19 0.0695 rpy=0 -0 0
- joint r_hip_yaw: origin xyz=0 1.68519e-34 -0.0665 rpy=-1.5708 -6.16298e-33 6.12323e-17 -> xyz=0 0 -0.0665 rpy=-1.5708 -6.16298e-33 6.12323e-17
- joint r_knee: origin xyz=-0.0009175 -0.234545 1.43617e-17 rpy=3.14159 -1.2326e-32 1.5708 -> xyz=0 -0.2236 1.36916e-17 rpy=3.14159 -1.2326e-32 1.5708
- joint r_sole_fixed_joint: origin xyz=0 0 0.075 rpy=0 1.5708 0 -> xyz=-0.0353 -1.38778e-17 -0.001 rpy=3.14159 -0 0

Commit message: [iCubParis*][conf] fix ft sensor position in the ankle

File: app/robots/iCubParis01/model.urdf (robot description, URDF)
Before this commit: robot test_icub, 55 links, 54 joints
Links:
- link neck_1: mass 0 -> 0.270176
- link neck_2: mass 0 -> 0.272306
Joints:
- joint codyco_balancing_world_fixed_joint: origin xyz=-0.0353 -1.38778e-17 -0.001 rpy=3.14159 -0 0 -> xyz=-0.0353 -7.60894e-35 -0.001 rpy=3.14159 -0 0
- joint imu_frame_fixed_joint: origin xyz=0.0185 -0.1108 0.0066 rpy=1.5708 -0 0 -> xyz=0.0225 -0.1005 0.0066 rpy=1.5708 -0 0
- joint l_foot_ft_sensor: origin xyz=0.0135 0 0.0695 rpy=0 -0 0 -> xyz=0.017 0 0.042 rpy=0 -0 0
- joint l_sole_fixed_joint: origin xyz=-0.0353 -1.38778e-17 -0.001 rpy=3.14159 -0 0 -> xyz=-0.0353 -7.60894e-35 -0.001 rpy=3.14159 -0 0
- joint neck_roll: origin xyz=0.0095 0 0 rpy=-1.5708 -0 -1.5708 -> xyz=0.033 -2.13821e-50 0 rpy=-1.5708 -0 -1.5708
- joint neck_yaw: origin xyz=-5.77779e-34 0 0 rpy=-1.5708 -0 1.5708 -> xyz=0 -0.001 0 rpy=-1.5708 -0 1.5708
- joint r_foot_ft_sensor: origin xyz=0.0135 4.28626e-19 0.0695 rpy=0 -0 0 -> xyz=0.017 0 0.042 rpy=0 -0 0

File: app/robots/iCubParis02/model.urdf (robot description, URDF)
Before this commit: robot test_icub, 55 links, 54 joints
Joints:
- joint codyco_balancing_world_fixed_joint: origin xyz=-0.0353 -1.38778e-17 -0.001 rpy=3.14159 -0 0 -> xyz=-0.0263 -5.66898e-35 -0.0143 rpy=3.14159 -0 0
- joint l_foot_dh_frame_fixed_joint: origin xyz=-0.0353 0 -0.001 rpy=0 1.5708 0 -> xyz=-0.0263 0 -0.0143 rpy=0 1.5708 0
- joint l_foot_ft_sensor: origin xyz=0.0135 0 0.0695 rpy=0 -0 0 -> xyz=0.008 0 0.0553 rpy=0 -0 0
- joint l_sole_fixed_joint: origin xyz=-0.0353 -1.38778e-17 -0.001 rpy=3.14159 -0 0 -> xyz=-0.0263 -5.66898e-35 -0.0143 rpy=3.14159 -0 0
- joint r_foot_dh_frame_fixed_joint: origin xyz=-0.0353 0 -0.001 rpy=0 1.5708 0 -> xyz=-0.0263 0 -0.0143 rpy=0 1.5708 0
- joint r_foot_ft_sensor: origin xyz=0.0135 4.28626e-19 0.0695 rpy=0 -0 0 -> xyz=0.008 0 0.0553 rpy=0 -0 0
- joint r_sole_fixed_joint: origin xyz=-0.0353 -1.38778e-17 -0.001 rpy=3.14159 -0 0 -> xyz=-0.0263 -1.38778e-17 -0.0143 rpy=3.14159 -0 0
