Commit message: update and refresh configuration files for iCubGenova*

File: app/robots/iCubGenova01/model.urdf (robot description, URDF)
Before this commit: robot test_icub, 46 links, 45 joints
Links:
- link l_ankle_1: mass 0.746 -> 0.643
- link l_hip_1: mass 0.754 -> 0.695
- link l_hip_2: mass 0.526 -> 0.982
- link l_leg: mass 1.264 -> 2.032
- link l_thigh: mass 2.175 -> 1.522
- link r_ankle_1: mass 0.746 -> 0.643
- link r_hip_1: mass 0.754 -> 0.695
- link r_hip_2: mass 0.526 -> 0.982
- link r_leg: mass 1.264 -> 2.032
- link r_thigh: mass 2.175 -> 1.522
Joints:
- joint l_ankle_pitch: origin xyz=-0.213 0 0 rpy=-1.5708 0 0 -> xyz=-0.2005 0 0 rpy=-1.5708 0 0
- joint l_hip_yaw: origin xyz=0 0 0 rpy=1.5708 -0 -1.5708 -> xyz=1.68519e-34 0 0 rpy=1.5708 -0 -1.5708
- joint l_knee: origin xyz=0 -0.2236 -1.36916e-17 rpy=3.14159 -1.2326e-32 1.5708 -> xyz=-0.0009175 -0.234545 -1.43617e-17 rpy=3.14159 -1.2326e-32 1.5708
- joint r_ankle_pitch: origin xyz=-0.213 0 0 rpy=1.5708 -0 0 -> xyz=-0.2005 0 0 rpy=1.5708 -0 0
- joint r_hip_yaw: origin xyz=0 0 0 rpy=-1.5708 -0 -1.5708 -> xyz=1.68519e-34 0 0 rpy=-1.5708 -0 -1.5708
- joint r_knee: origin xyz=0 -0.2236 1.36916e-17 rpy=3.14159 -1.2326e-32 1.5708 -> xyz=-0.0009175 -0.234545 1.43617e-17 rpy=3.14159 -1.2326e-32 1.5708

Commit message: Update iCubGenova* and iCubParis* to contain the chest_skin_frame

File: app/robots/iCubGenova01/model.urdf (robot description, URDF)
Before this commit: robot test_icub, 55 links, 54 joints
Links:
- added link chest_skin_frame, mass 0
- link l_ankle_2: mass 0.1 -> 0.2675
- link l_foot: mass 0.761 -> 0.5935
- link r_ankle_2: mass 0.1 -> 0.2675
- link r_foot: mass 0.761 -> 0.5935
Joints:
- added joint chest_skin_frame_fixed_joint: type fixed, parent chest, child chest_skin_frame, origin xyz=0.00231 0.1933 -1.18362e-17 rpy=-1.8747e-33 5.77686e-66 6.16298e-33, axis 0 0 0
- joint codyco_balancing_world_fixed_joint: origin xyz=-8.67362e-19 -1.38778e-17 0.075 rpy=3.14159 -0 0 -> xyz=-8.67362e-19 -1.38778e-17 0.004 rpy=3.14159 -0 0
- joint l_foot_dh_frame_fixed_joint: origin xyz=-8.67362e-19 -1.38778e-17 0.075 rpy=-9.70754e-18 1.5708 -9.70754e-18 -> xyz=0 0 0.004 rpy=0 1.5708 0
- joint l_foot_ft_sensor: origin xyz=-0.0035 0 -0.0065 rpy=0 -0 0 -> xyz=-0.0035 0 0.0645 rpy=0 -0 0
- joint l_sole_fixed_joint: origin xyz=0 0 0.075 rpy=0 1.5708 0 -> xyz=-8.67362e-19 -1.38778e-17 0.004 rpy=3.14159 -0 0
- joint r_foot_dh_frame_fixed_joint: origin xyz=-8.67362e-19 1.38778e-17 0.075 rpy=-1.01315e-16 1.5708 -1.01315e-16 -> xyz=0 0 0.004 rpy=0 1.5708 0
- joint r_foot_ft_sensor: origin xyz=-0.0035 4.28626e-19 -0.0065 rpy=0 -0 0 -> xyz=-0.0035 4.28626e-19 0.0645 rpy=0 -0 0
- joint r_sole_fixed_joint: origin xyz=0 0 0.075 rpy=0 1.5708 0 -> xyz=-8.67362e-19 1.38778e-17 0.004 rpy=3.14159 -0 0

File: app/robots/iCubGenova03/model.urdf (robot description, URDF)
Before this commit: robot test_icub, 55 links, 54 joints
Links:
- added link chest_skin_frame, mass 0
- link l_ankle_2: mass 0.1 -> 0.2675
- link l_foot: mass 0.761 -> 0.5935
- link r_ankle_2: mass 0.1 -> 0.2675
- link r_foot: mass 0.761 -> 0.5935
Joints:
- added joint chest_skin_frame_fixed_joint: type fixed, parent chest, child chest_skin_frame, origin xyz=0.00231 0.1933 -1.18362e-17 rpy=-1.8747e-33 5.77686e-66 6.16298e-33, axis 0 0 0
- joint codyco_balancing_world_fixed_joint: origin xyz=-1.84889e-33 -1.38778e-17 0.075 rpy=3.14159 -0 0 -> xyz=-0.0353 -7.60894e-35 -0.001 rpy=3.14159 -0 0
- joint l_foot_dh_frame_fixed_joint: origin xyz=-1.84889e-33 -1.38778e-17 0.075 rpy=-9.70754e-18 1.5708 -9.70754e-18 -> xyz=-0.0353 0 -0.001 rpy=0 1.5708 0
- joint l_foot_ft_sensor: origin xyz=-0.0035 0 -0.0065 rpy=0 -0 0 -> xyz=0.017 0 0.042 rpy=0 -0 0
- joint l_sole_fixed_joint: origin xyz=0 0 0.075 rpy=0 1.5708 0 -> xyz=-0.0353 -7.60894e-35 -0.001 rpy=3.14159 -0 0
- joint r_foot_dh_frame_fixed_joint: origin xyz=-8.67362e-19 1.38778e-17 0.075 rpy=-1.01315e-16 1.5708 -1.01315e-16 -> xyz=-0.0353 0 -0.001 rpy=0 1.5708 0
- joint r_foot_ft_sensor: origin xyz=-0.0035 4.28626e-19 -0.0065 rpy=0 -0 0 -> xyz=0.017 0 0.042 rpy=0 -0 0
- joint r_sole_fixed_joint: origin xyz=0 0 0.075 rpy=0 1.5708 0 -> xyz=-0.0353 -1.38778e-17 -0.001 rpy=3.14159 -0 0

File: app/robots/iCubParis01/model.urdf (robot description, URDF)
Before this commit: robot iCub, 55 links, 54 joints
Links:
- added link chest_skin_frame, mass 0
Joints:
- added joint chest_skin_frame_fixed_joint: type fixed, parent chest, child chest_skin_frame, origin xyz=0.00231 0.1933 -1.18362e-17 rpy=-1.8747e-33 5.77686e-66 6.16298e-33, axis 0 0 0

File: app/robots/iCubParis02/model.urdf (robot description, URDF)
Before this commit: robot iCub, 55 links, 54 joints
Links:
- added link chest_skin_frame, mass 0
Joints:
- added joint chest_skin_frame_fixed_joint: type fixed, parent chest, child chest_skin_frame, origin xyz=0.00231 0.1933 -1.18362e-17 rpy=-1.8747e-33 5.77686e-66 6.16298e-33, axis 0 0 0
