Commit message: Added r_foot_dh_frame and l_foot_dh_frame to iCubGenova02 nobattery

File: app/robots/iCubGenova02/model_nobattery.urdf (robot description, URDF)
Before this commit: robot iCubGenova02, 103 links, 102 joints
Links:
- added link l_foot_dh_frame
- added link r_foot_dh_frame
Joints:
- added joint l_foot_dh_frame_fixed_joint: type fixed, parent l_foot, child l_foot_dh_frame, origin xyz=0.0 0 0.004 rpy=0 1.5708 0, axis 0 0 0
- added joint r_foot_dh_frame_fixed_joint: type fixed, parent r_foot, child r_foot_dh_frame, origin xyz=0.0 0 0.004 rpy=0 1.5708 0, axis 0 0 0
