Commit message: Added updated file for iCubGenova02

File: app/robots/iCubGenova02/model.urdf (robot description, URDF)
Before this commit: robot test_icub, 24 links, 23 joints
Links:
- removed link base_link
- removed link l_arm
- removed link r_arm
- added link l_shoulder_3, mass 0.156157
- added link r_shoulder_3, mass 0.155
- link l_upper_arm: mass 0.156157 -> 0.727843; geometry collision mesh filename=meshes/collision/icub_simple_collision_l_arm.dae scale=1 1 1; visual mesh filename=meshes/visual/icub_l_arm.dae scale=1 1 1
- link r_upper_arm: mass 0.155 -> 0.729; geometry collision mesh filename=meshes/collision/icub_simple_collision_r_arm.dae scale=1 1 1; visual mesh filename=meshes/visual/icub_r_arm.dae scale=1 1 1
Joints:
- removed joint base_fixed_joint
- joint l_arm_ft_sensor: child l_arm -> l_upper_arm; origin xyz=0.015 9.36797e-18 0.15228 rpy=-1.5708 0 0 -> xyz=0.015 9.36797e-18 0.068 rpy=0 -0 0; parent l_upper_arm -> l_shoulder_3
- joint l_elbow: origin xyz=0 0 0 rpy=1.5708 -0 0 -> xyz=0 0 0.08428 rpy=-6.12323e-17 0 0; parent l_arm -> l_upper_arm
- joint l_shoulder_yaw: child l_upper_arm -> l_shoulder_3
- joint r_arm_ft_sensor: child r_arm -> r_upper_arm; origin xyz=0.015 -8.93429e-18 0.15228 rpy=1.5708 -0 3.14159 -> xyz=0.015 -8.93429e-18 0.068 rpy=0 -0 0; parent r_upper_arm -> r_shoulder_3
- joint r_elbow: origin xyz=0 0 0 rpy=1.5708 -0 0 -> xyz=0 0 0.08428 rpy=3.14159 -0 3.14159; parent r_arm -> r_upper_arm
- joint r_shoulder_yaw: child r_upper_arm -> r_shoulder_3

File: app/robots/iCubGenova02/model_noleftarm.urdf (robot description, URDF)
Before this commit: robot test_icub, 15 links, 14 joints
Links:
- removed link base_link
- removed link r_arm
- added link r_shoulder_3, mass 0.155
- link r_upper_arm: mass 0.155 -> 0.729; geometry collision mesh filename=meshes/collision/icub_simple_collision_r_arm.dae scale=1 1 1; visual mesh filename=meshes/visual/icub_r_arm.dae scale=1 1 1
Joints:
- removed joint base_fixed_joint
- joint r_arm_ft_sensor: child r_arm -> r_upper_arm; origin xyz=0.015 -8.93429e-18 0.15228 rpy=1.5708 -0 3.14159 -> xyz=0.015 -8.93429e-18 0.068 rpy=0 -0 0; parent r_upper_arm -> r_shoulder_3
- joint r_elbow: origin xyz=0 0 0 rpy=1.5708 -0 0 -> xyz=0 0 0.08428 rpy=3.14159 -0 3.14159; parent r_arm -> r_upper_arm
- joint r_shoulder_yaw: child r_upper_arm -> r_shoulder_3

Commit message: Add new model for iCubGenova02, accounting for the backpack. No reliable backpack information was available, so we estimated the mass of the backpack to be ~1.5 kg and we moved the COM of the chest 2.3 cm in the back. We still are ignoring the known offset in the arms.

File: app/robots/iCubGenova02/model.urdf (robot description, URDF)
Before this commit: robot test_icub, 23 links, 22 joints
Links:
- added link base_link
- added link chest_skin_frame, mass 0
- added link codyco_balancing_world, mass 0
- added link l_ankle_1, mass 0.643; collision mesh filename=meshes/collision/icub_simple_collision_l_ankle_1.dae scale=1 1 1; visual mesh filename=meshes/visual/icub_l_ankle_1.dae scale=1 1 1
- added link l_ankle_2, mass 0.2675
- added link l_foot, mass 0.5935; collision mesh filename=meshes/collision/icub_simple_collision_l_foot.dae scale=1 1 1; visual mesh filename=meshes/visual/icub_l_foot.dae scale=1 1 1
- added link l_foot_dh_frame, mass 0
- added link l_forearm_dh_frame, mass 0
- added link l_hand_dh_frame, mass 0
- added link l_hip_1, mass 0.695; collision mesh filename=meshes/collision/icub_simple_collision_l_hip_1.dae scale=1 1 1; visual mesh filename=meshes/visual/icub_l_hip_1.dae scale=1 1 1
- added link l_hip_2, mass 0.982; collision mesh filename=meshes/collision/icub_simple_collision_l_hip_2.dae scale=1 1 1; visual mesh filename=meshes/visual/icub_l_hip_2.dae scale=1 1 1
- added link l_hip_3, mass 0
- added link l_lower_leg, mass 2.032; collision mesh filename=meshes/collision/icub_simple_collision_l_shank.dae scale=1 1 1; visual mesh filename=meshes/visual/icub_l_shank.dae scale=1 1 1
- added link l_sole, mass 0
- added link l_upper_arm_dh_frame, mass 0
- added link l_upper_leg, mass 1.522; collision mesh filename=meshes/collision/icub_simple_collision_l_thigh.dae scale=1 1 1; visual mesh filename=meshes/visual/icub_l_thigh.dae scale=1 1 1
- added link r_ankle_1, mass 0.643; collision mesh filename=meshes/collision/icub_simple_collision_r_ankle_1.dae scale=1 1 1; visual mesh filename=meshes/visual/icub_r_ankle_1.dae scale=1 1 1
- added link r_ankle_2, mass 0.2675
- added link r_foot, mass 0.5935; collision mesh filename=meshes/collision/icub_simple_collision_r_foot.dae scale=1 1 1; visual mesh filename=meshes/visual/icub_r_foot.dae scale=1 1 1
- added link r_foot_dh_frame, mass 0
- added link r_forearm_dh_frame, mass 0
- added link r_hand_dh_frame, mass 0
- added link r_hip_1, mass 0.695; collision mesh filename=meshes/collision/icub_simple_collision_r_hip_1.dae scale=1 1 1; visual mesh filename=meshes/visual/icub_r_hip_1.dae scale=1 1 1
- added link r_hip_2, mass 0.982; collision mesh filename=meshes/collision/icub_simple_collision_r_hip_2.dae scale=1 1 1; visual mesh filename=meshes/visual/icub_r_hip_2.dae scale=1 1 1
- added link r_hip_3, mass 0
- added link r_lower_leg, mass 2.032; collision mesh filename=meshes/collision/icub_simple_collision_r_shank.dae scale=1 1 1; visual mesh filename=meshes/visual/icub_r_shank.dae scale=1 1 1
- added link r_sole, mass 0
- added link r_upper_arm_dh_frame, mass 0
- added link r_upper_leg, mass 1.522; collision mesh filename=meshes/collision/icub_simple_collision_r_thigh.dae scale=1 1 1; visual mesh filename=meshes/visual/icub_r_thigh.dae scale=1 1 1
- added link root_link, mass 4.72; collision mesh filename=meshes/collision/icub_simple_collision_root_link.dae scale=1 1 1; visual mesh filename=meshes/visual/icub_root_link.dae scale=1 1 1
- added link torso, mass 0
- added link torso_1, mass 0; collision mesh filename=meshes/collision/icub_simple_collision_lap_belt_1.dae scale=1 1 1; visual mesh filename=meshes/visual/icub_lap_belt_1.dae scale=1 1 1
- added link torso_2, mass 0
- link chest: mass 4.81 -> 6.31
Joints:
- added joint base_fixed_joint: type fixed, parent base_link, child root_link, origin xyz=0 0 0 rpy=0 -0 0, axis 0 0 0
- added joint chest_skin_frame_fixed_joint: type fixed, parent chest, child chest_skin_frame, origin xyz=0.00231 0.1933 -1.18362e-17 rpy=-1.8747e-33 5.77686e-66 6.16298e-33, axis 0 0 0
- added joint codyco_balancing_world_fixed_joint: type fixed, parent l_foot, child codyco_balancing_world, origin xyz=-8.67362e-19 -1.38778e-17 0.004 rpy=3.14159 -0 0, axis 0 0 0
- added joint l_ankle_pitch: type revolute, parent l_lower_leg, child l_ankle_1, origin xyz=-0.2005 0 0 rpy=-1.5708 0 0, axis 0 -1 6.12323e-17, limit lower=-0.733038 upper=0.366519 effort=24 velocity=100
- added joint l_ankle_roll: type revolute, parent l_ankle_1, child l_ankle_2, origin xyz=0 0 0 rpy=0 -1.5708 0, axis 1 0 0, limit lower=-0.418879 upper=0.418879 effort=11 velocity=100
- added joint l_foot_dh_frame_fixed_joint: type fixed, parent l_foot, child l_foot_dh_frame, origin xyz=0 0 0.004 rpy=0 1.5708 0, axis 0 0 0
- added joint l_foot_ft_sensor: type fixed, parent l_ankle_2, child l_foot, origin xyz=-0.0035 0 0.0645 rpy=0 -0 0, axis 0 0 0
- added joint l_forearm_dh_frame_fixed_joint: type fixed, parent l_forearm, child l_forearm_dh_frame, origin xyz=0 0.1373 8.4072e-18 rpy=0 -0 0, axis 0 0 0
- added joint l_hand_dh_frame_fixed_joint: type fixed, parent l_hand, child l_hand_dh_frame, origin xyz=0.0625 0 -0.016 rpy=0 -0 0, axis 0 0 0
- added joint l_hip_pitch: type revolute, parent root_link, child l_hip_1, origin xyz=0 -0.0681 -0.1199 rpy=-3.14159 1.5708 -2.77556e-17, axis 0 -1 6.12323e-17, limit lower=-0.767945 upper=2.30383 effort=84 velocity=100
- added joint l_hip_roll: type revolute, parent l_hip_1, child l_hip_2, origin xyz=0 0 0 rpy=3.14159 -1.5708 -2.77556e-17, axis 1 0 -6.12323e-17, limit lower=-2.07694 upper=0.296706 effort=84 velocity=100
- added joint l_hip_yaw: type revolute, parent l_hip_3, child l_upper_leg, origin xyz=0 -1.68519e-34 -0.0665 rpy=-1.5708 -6.16298e-33 -6.12323e-17, axis 0 1 6.12323e-17, limit lower=-1.37881 upper=1.37881 effort=40 velocity=100
- added joint l_knee: type revolute, parent l_upper_leg, child l_lower_leg, origin xyz=-0.0009175 -0.234545 -1.43617e-17 rpy=3.14159 -1.2326e-32 1.5708, axis 0 1.22465e-16 -1, limit lower=-2.18166 upper=0.401426 effort=30 velocity=100
- added joint l_leg_ft_sensor: type fixed, parent l_hip_2, child l_hip_3, origin xyz=0 0 0.0665 rpy=0 -0 0, axis 0 0 0
- added joint l_sole_fixed_joint: type fixed, parent l_foot, child l_sole, origin xyz=-8.67362e-19 -1.38778e-17 0.004 rpy=3.14159 -0 0, axis 0 0 0
- added joint l_upper_arm_dh_frame_fixed_joint: type fixed, parent l_upper_arm, child l_upper_arm_dh_frame, origin xyz=0 0 0.08428 rpy=-1.5708 0 0, axis 0 0 0
- added joint r_ankle_pitch: type revolute, parent r_lower_leg, child r_ankle_1, origin xyz=-0.2005 0 0 rpy=1.5708 -0 0, axis 0 1 6.12323e-17, limit lower=-0.733038 upper=0.366519 effort=24 velocity=100
- added joint r_ankle_roll: type revolute, parent r_ankle_1, child r_ankle_2, origin xyz=0 0 0 rpy=0.504019 1.5708 -2.63757, axis -1 1.22465e-16 0, limit lower=-0.418879 upper=0.418879 effort=11 velocity=100
- added joint r_foot_dh_frame_fixed_joint: type fixed, parent r_foot, child r_foot_dh_frame, origin xyz=0 0 0.004 rpy=0 1.5708 0, axis 0 0 0
- added joint r_foot_ft_sensor: type fixed, parent r_ankle_2, child r_foot, origin xyz=-0.0035 4.28626e-19 0.0645 rpy=0 -0 0, axis 0 0 0
- added joint r_forearm_dh_frame_fixed_joint: type fixed, parent r_forearm, child r_forearm_dh_frame, origin xyz=0 -0.1373 -8.4072e-18 rpy=0 -0 0, axis 0 0 0
- added joint r_hand_dh_frame_fixed_joint: type fixed, parent r_hand, child r_hand_dh_frame, origin xyz=0.0625 0 0.016 rpy=0 -0 0, axis 0 0 0
- added joint r_hip_pitch: type revolute, parent root_link, child r_hip_1, origin xyz=0 0.0681 -0.1199 rpy=-2.77556e-17 1.5708 2.77556e-17, axis 0 1 6.12323e-17, limit lower=-0.767945 upper=2.30383 effort=84 velocity=100
- added joint r_hip_roll: type revolute, parent r_hip_1, child r_hip_2, origin xyz=0 0 0 rpy=2.77556e-17 1.5708 -2.77556e-17, axis -1 0 6.12323e-17, limit lower=-2.07694 upper=0.296706 effort=84 velocity=100
- added joint r_hip_yaw: type revolute, parent r_hip_3, child r_upper_leg, origin xyz=0 1.68519e-34 -0.0665 rpy=-1.5708 -6.16298e-33 6.12323e-17, axis 0 -1 6.12323e-17, limit lower=-1.37881 upper=1.37881 effort=40 velocity=100
- added joint r_knee: type revolute, parent r_upper_leg, child r_lower_leg, origin xyz=-0.0009175 -0.234545 1.43617e-17 rpy=3.14159 -1.2326e-32 1.5708, axis 0 1.22465e-16 -1, limit lower=-2.18166 upper=0.401426 effort=30 velocity=100
- added joint r_leg_ft_sensor: type fixed, parent r_hip_2, child r_hip_3, origin xyz=0 0 0.0665 rpy=0 -0 0, axis 0 0 0
- added joint r_sole_fixed_joint: type fixed, parent r_foot, child r_sole, origin xyz=-8.67362e-19 1.38778e-17 0.004 rpy=3.14159 -0 0, axis 0 0 0
- added joint r_upper_arm_dh_frame_fixed_joint: type fixed, parent r_upper_arm, child r_upper_arm_dh_frame, origin xyz=0 0 0.08428 rpy=1.5708 -0 3.14159, axis 0 0 0
- added joint torso_joint: type fixed, parent chest, child torso, origin xyz=0.00231 0.1933 -1.18362e-17 rpy=0 -0 0, axis 0 0 0
- added joint torso_pitch: type revolute, parent root_link, child torso_1, origin xyz=0 0 0 rpy=-2.77556e-17 -1.5708 3.14159, axis 0 1 6.12323e-17, limit lower=-0.383972 upper=1.46608 effort=36 velocity=100
- added joint torso_roll: type revolute, parent torso_1, child torso_2, origin xyz=0.032 -2.67276e-51 0 rpy=1.5708 -0 -1.5708, axis 0 1 6.12323e-17, limit lower=-0.680678 upper=0.680678 effort=80 velocity=100
- added joint torso_yaw: type revolute, parent torso_2, child chest, origin xyz=-7.46298e-34 -0.0055 0 rpy=-1.5708 -0 -1.5708, axis 0 -1 6.12323e-17, limit lower=-1.02974 upper=1.02974 effort=80 velocity=100
