Commit message: Fixed axis of rotation of torso_roll
cc @traversaro @fiorisi @DanielePucci

File: app/robots/iCubGenova02/model.urdf (robot description, URDF)
Before this commit: robot iCubGenova02, 103 links, 102 joints
Joints:
- joint torso_roll: axis 0.0 0.0 1.0 -> 0.0 0.0 -1.0

File: app/robots/iCubGenova02/model_nobattery.urdf (robot description, URDF)
Before this commit: robot iCubGenova02, 105 links, 104 joints
Joints:
- joint torso_roll: axis 0.0 0.0 1.0 -> 0.0 0.0 -1.0
