Commit message: [iCubGenova02] Import model with wrist dofs from icub-model-generator

File: app/robots/iCubGenova02/model.urdf (robot description, URDF)
Before this commit: robot iCubGenova02, 105 links, 104 joints
Links:
- added link l_forearm, mass 0.636185; collision mesh filename=model://iCubGenova02/meshes/dae/sim_sea_2-5_l_forearm_prt.d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 scale=0.001 0.001 0.001; visual mesh filename=model://iCubGenova02/meshes/dae/sim_sea_2-5_l_forearm_prt.d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 scale=0.001 0.001 0.001
- added link l_forearm_dh_frame
- added link l_forearm_skin_0
- added link l_forearm_skin_1
- added link l_forearm_skin_10
- added link l_forearm_skin_11
- added link l_forearm_skin_12
- added link l_forearm_skin_13
- added link l_forearm_skin_14
- added link l_forearm_skin_15
- added link l_forearm_skin_16
- added link l_forearm_skin_17
- added link l_forearm_skin_19
- added link l_forearm_skin_2
- added link l_forearm_skin_22
- added link l_forearm_skin_24
- added link l_forearm_skin_25
- added link l_forearm_skin_28
- added link l_forearm_skin_29
- added link l_forearm_skin_3
- added link l_forearm_skin_4
- added link l_forearm_skin_5
- added link l_forearm_skin_6
- added link l_forearm_skin_7
- added link l_forearm_skin_8
- added link l_forearm_skin_9
- added link l_hand, mass 0.247806; collision mesh filename=model://iCubGenova02/meshes/dae/sim_sea_2-5_l_hand_prt.dae scale=0.001 0.001 0.001; visual mesh filename=model://iCubGenova02/meshes/dae/sim_sea_2-5_l_hand_prt.dae scale=0.001 0.001 0.001
- added link l_hand_dh_frame
- added link l_wrist_1, mass 0.0362152; collision mesh filename=model://iCubGenova02/meshes/dae/sim_sea_2-5_l_wrist_pitch_p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 scale=0.001 0.001 0.001; visual mesh filename=model://iCubGenova02/meshes/dae/sim_sea_2-5_l_wrist_pitch_p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 scale=0.001 0.001 0.001
- added link r_forearm, mass 0.6347; collision mesh filename=model://iCubGenova02/meshes/dae/sim_sea_2-5_r_forearm_prt.d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 scale=0.001 0.001 0.001; visual mesh filename=model://iCubGenova02/meshes/dae/sim_sea_2-5_r_forearm_prt.d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 scale=0.001 0.001 0.001
- added link r_forearm_dh_frame
- added link r_forearm_skin_0
- added link r_forearm_skin_1
- added link r_forearm_skin_10
- added link r_forearm_skin_11
- added link r_forearm_skin_12
- added link r_forearm_skin_13
- added link r_forearm_skin_14
- added link r_forearm_skin_15
- added link r_forearm_skin_16
- added link r_forearm_skin_17
- added link r_forearm_skin_19
- added link r_forearm_skin_2
- added link r_forearm_skin_22
- added link r_forearm_skin_24
- added link r_forearm_skin_25
- added link r_forearm_skin_28
- added link r_forearm_skin_29
- added link r_forearm_skin_3
- added link r_forearm_skin_4
- added link r_forearm_skin_5
- added link r_forearm_skin_6
- added link r_forearm_skin_7
- added link r_forearm_skin_8
- added link r_forearm_skin_9
- added link r_hand, mass 0.248289; collision mesh filename=model://iCubGenova02/meshes/dae/sim_sea_2-5_r_hand_prt.dae scale=0.001 0.001 0.001; visual mesh filename=model://iCubGenova02/meshes/dae/sim_sea_2-5_r_hand_prt.dae scale=0.001 0.001 0.001
- added link r_hand_dh_frame
- added link r_wrist_1, mass 0.0362615; collision mesh filename=model://iCubGenova02/meshes/dae/sim_sea_2-5_r_wrist_pitch_p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 scale=0.001 0.001 0.001; visual mesh filename=model://iCubGenova02/meshes/dae/sim_sea_2-5_r_wrist_pitch_p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 scale=0.001 0.001 0.001
- link chest: geometry collision mesh filename=model://iCubGenova02/meshes/dae/sim_sea_2-5_chest_bb_prt.dae scale=0.001 0.001 0.001; visual mesh filename=model://iCubGenova02/meshes/dae/sim_sea_2-5_chest_bb_prt.dae scale=0.001 0.001 0.001
- link head: geometry collision mesh filename=model://iCubGenova02/meshes/dae/sim_sea_2-5_head_prt.dae scale=0.001 0.001 0.001; visual mesh filename=model://iCubGenova02/meshes/dae/sim_sea_2-5_head_prt.dae scale=0.001 0.001 0.001
- link l_ankle_1: geometry collision mesh filename=model://iCubGenova02/meshes/dae/sim_sea_2-5_l_ankle_prt.dae scale=0.001 0.001 0.001; visual mesh filename=model://iCubGenova02/meshes/dae/sim_sea_2-5_l_ankle_prt.dae scale=0.001 0.001 0.001
- link l_ankle_2: geometry collision mesh filename=model://iCubGenova02/meshes/dae/sim_sea_2-5_l_foot_prt.dae scale=0.001 0.001 0.001; visual mesh filename=model://iCubGenova02/meshes/dae/sim_sea_2-5_l_foot_prt.dae scale=0.001 0.001 0.001
- link l_elbow_1: mass 1.17718 -> 0.267903; geometry collision mesh filename=model://iCubGenova02/meshes/dae/sim_sea_2-5_l_elbow_prosup_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 scale=0.001 0.001 0.001; visual mesh filename=model://iCubGenova02/meshes/dae/sim_sea_2-5_l_elbow_prosup_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 scale=0.001 0.001 0.001
- link l_foot: geometry collision mesh filename=model://iCubGenova02/meshes/dae/sim_sea_2-5_l_sole_prt.dae scale=0.001 0.001 0.001; visual mesh filename=model://iCubGenova02/meshes/dae/sim_sea_2-5_l_sole_prt.dae scale=0.001 0.001 0.001
- link l_hip_1: geometry collision mesh filename=model://iCubGenova02/meshes/dae/sim_sea_2-5_l_hip_1_prt.dae scale=0.001 0.001 0.001; visual mesh filename=model://iCubGenova02/meshes/dae/sim_sea_2-5_l_hip_1_prt.dae scale=0.001 0.001 0.001
- link l_hip_2: geometry collision mesh filename=model://iCubGenova02/meshes/dae/sim_sea_2-5_l_hip_2_prt.dae scale=0.001 0.001 0.001; visual mesh filename=model://iCubGenova02/meshes/dae/sim_sea_2-5_l_hip_2_prt.dae scale=0.001 0.001 0.001
- link l_hip_3: geometry collision mesh filename=model://iCubGenova02/meshes/dae/sim_sea_2-5_l_upper_thigh_p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 scale=0.001 0.001 0.001; visual mesh filename=model://iCubGenova02/meshes/dae/sim_sea_2-5_l_upper_thigh_p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 scale=0.001 0.001 0.001
- link l_lower_leg: geometry collision mesh filename=model://iCubGenova02/meshes/dae/sim_sea_2-5_l_shank_prt.dae scale=0.001 0.001 0.001; visual mesh filename=model://iCubGenova02/meshes/dae/sim_sea_2-5_l_shank_prt.dae scale=0.001 0.001 0.001
- link l_shoulder_1: geometry collision mesh filename=model://iCubGenova02/meshes/dae/sim_sea_2-5_l_shoulder_1_pr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 scale=0.001 0.001 0.001; visual mesh filename=model://iCubGenova02/meshes/dae/sim_sea_2-5_l_shoulder_1_pr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 scale=0.001 0.001 0.001
- link l_shoulder_2: mass 0.239074 -> 0.238162; geometry collision mesh filename=model://iCubGenova02/meshes/dae/sim_sea_2-5_l_shoulder_2_pr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 scale=0.001 0.001 0.001; visual mesh filename=model://iCubGenova02/meshes/dae/sim_sea_2-5_l_shoulder_2_pr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 scale=0.001 0.001 0.001
- link l_shoulder_3: geometry collision mesh filename=model://iCubGenova02/meshes/dae/sim_sea_2-5_l_upper_arm_prt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 scale=0.001 0.001 0.001; visual mesh filename=model://iCubGenova02/meshes/dae/sim_sea_2-5_l_upper_arm_prt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 scale=0.001 0.001 0.001
- link l_upper_arm: geometry collision mesh filename=model://iCubGenova02/meshes/dae/sim_sea_2-5_l_elbow_prt.dae scale=0.001 0.001 0.001; visual mesh filename=model://iCubGenova02/meshes/dae/sim_sea_2-5_l_elbow_prt.dae scale=0.001 0.001 0.001
- link l_upper_leg: geometry collision mesh filename=model://iCubGenova02/meshes/dae/sim_sea_2-5_l_thigh_prt.dae scale=0.001 0.001 0.001; visual mesh filename=model://iCubGenova02/meshes/dae/sim_sea_2-5_l_thigh_prt.dae scale=0.001 0.001 0.001
- link neck_1: geometry collision mesh filename=model://iCubGenova02/meshes/dae/sim_sea_2-5_neck_1_prt.dae scale=0.001 0.001 0.001; visual mesh filename=model://iCubGenova02/meshes/dae/sim_sea_2-5_neck_1_prt.dae scale=0.001 0.001 0.001
- link neck_2: geometry collision mesh filename=model://iCubGenova02/meshes/dae/sim_sea_2-5_neck_2_prt.dae scale=0.001 0.001 0.001; visual mesh filename=model://iCubGenova02/meshes/dae/sim_sea_2-5_neck_2_prt.dae scale=0.001 0.001 0.001
- link r_ankle_1: geometry collision mesh filename=model://iCubGenova02/meshes/dae/sim_sea_2-5_r_ankle_prt.dae scale=0.001 0.001 0.001; visual mesh filename=model://iCubGenova02/meshes/dae/sim_sea_2-5_r_ankle_prt.dae scale=0.001 0.001 0.001
- link r_ankle_2: geometry collision mesh filename=model://iCubGenova02/meshes/dae/sim_sea_2-5_r_foot_prt.dae scale=0.001 0.001 0.001; visual mesh filename=model://iCubGenova02/meshes/dae/sim_sea_2-5_r_foot_prt.dae scale=0.001 0.001 0.001
- link r_elbow_1: mass 1.17637 -> 0.267903; geometry collision mesh filename=model://iCubGenova02/meshes/dae/sim_sea_2-5_r_elbow_prosup_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 scale=0.001 0.001 0.001; visual mesh filename=model://iCubGenova02/meshes/dae/sim_sea_2-5_r_elbow_prosup_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 scale=0.001 0.001 0.001
- link r_foot: geometry collision mesh filename=model://iCubGenova02/meshes/dae/sim_sea_2-5_r_sole_prt.dae scale=0.001 0.001 0.001; visual mesh filename=model://iCubGenova02/meshes/dae/sim_sea_2-5_r_sole_prt.dae scale=0.001 0.001 0.001
- link r_hip_1: mass 0.920354 -> 0.920101; geometry collision mesh filename=model://iCubGenova02/meshes/dae/sim_sea_2-5_r_hip_1_prt.dae scale=0.001 0.001 0.001; visual mesh filename=model://iCubGenova02/meshes/dae/sim_sea_2-5_r_hip_1_prt.dae scale=0.001 0.001 0.001
- link r_hip_2: geometry collision mesh filename=model://iCubGenova02/meshes/dae/sim_sea_2-5_r_hip_2_prt.dae scale=0.001 0.001 0.001; visual mesh filename=model://iCubGenova02/meshes/dae/sim_sea_2-5_r_hip_2_prt.dae scale=0.001 0.001 0.001
- link r_hip_3: geometry collision mesh filename=model://iCubGenova02/meshes/dae/sim_sea_2-5_r_upper_thigh_p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 scale=0.001 0.001 0.001; visual mesh filename=model://iCubGenova02/meshes/dae/sim_sea_2-5_r_upper_thigh_p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 scale=0.001 0.001 0.001
- link r_lower_leg: geometry collision mesh filename=model://iCubGenova02/meshes/dae/sim_sea_2-5_r_shank_prt.dae scale=0.001 0.001 0.001; visual mesh filename=model://iCubGenova02/meshes/dae/sim_sea_2-5_r_shank_prt.dae scale=0.001 0.001 0.001
- link r_shoulder_1: geometry collision mesh filename=model://iCubGenova02/meshes/dae/sim_sea_2-5_r_shoulder_1_pr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 scale=0.001 0.001 0.001; visual mesh filename=model://iCubGenova02/meshes/dae/sim_sea_2-5_r_shoulder_1_pr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 scale=0.001 0.001 0.001
- link r_shoulder_2: geometry collision mesh filename=model://iCubGenova02/meshes/dae/sim_sea_2-5_r_shoulder_2_pr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 scale=0.001 0.001 0.001; visual mesh filename=model://iCubGenova02/meshes/dae/sim_sea_2-5_r_shoulder_2_pr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 scale=0.001 0.001 0.001
- link r_shoulder_3: geometry collision mesh filename=model://iCubGenova02/meshes/dae/sim_sea_2-5_r_upper_arm_prt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 scale=0.001 0.001 0.001; visual mesh filename=model://iCubGenova02/meshes/dae/sim_sea_2-5_r_upper_arm_prt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 scale=0.001 0.001 0.001
- link r_upper_arm: geometry collision mesh filename=model://iCubGenova02/meshes/dae/sim_sea_2-5_r_elbow_prt.dae scale=0.001 0.001 0.001; visual mesh filename=model://iCubGenova02/meshes/dae/sim_sea_2-5_r_elbow_prt.dae scale=0.001 0.001 0.001
- link r_upper_leg: geometry collision mesh filename=model://iCubGenova02/meshes/dae/sim_sea_2-5_r_thigh_prt.dae scale=0.001 0.001 0.001; visual mesh filename=model://iCubGenova02/meshes/dae/sim_sea_2-5_r_thigh_prt.dae scale=0.001 0.001 0.001
- link root_link: geometry collision mesh filename=model://iCubGenova02/meshes/dae/sim_sea_2-5_root_link_prt.d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 scale=0.001 0.001 0.001; visual mesh filename=model://iCubGenova02/meshes/dae/sim_sea_2-5_root_link_prt.d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 scale=0.001 0.001 0.001
- link torso_1: geometry collision mesh filename=model://iCubGenova02/meshes/dae/sim_sea_2-5_lap_belt_1_prt.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 scale=0.001 0.001 0.001; visual mesh filename=model://iCubGenova02/meshes/dae/sim_sea_2-5_lap_belt_1_prt.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 scale=0.001 0.001 0.001
- link torso_2: mass 0.428161 -> 0.425685; geometry collision mesh filename=model://iCubGenova02/meshes/dae/sim_sea_2-5_lap_belt_2_prt.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 scale=0.001 0.001 0.001; visual mesh filename=model://iCubGenova02/meshes/dae/sim_sea_2-5_lap_belt_2_prt.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 scale=0.001 0.001 0.001
Joints:
- removed joint imu_frame_fixed_joint
- added joint imu_fixed_joint: type fixed, parent head, child imu_frame, origin xyz=0.00950000019074 0.133444 0.0093 rpy=-1.57079632679 1.57079632679 0
- added joint l_forearm_dh_frame_fixed_joint: type fixed, parent l_forearm, child l_forearm_dh_frame, origin xyz=0.102871102373 7.00000000002e-06 0.0275642213111 rpy=2.87979333376 0 1.57079632679
- added joint l_forearm_skin_0_fixed_joint: type fixed, parent l_forearm, child l_forearm_skin_0, origin xyz=0.0454493286618 -0.0323169 -0.00628656037901 rpy=1.69181522292 -0.271026744341 0.0727882713185
- added joint l_forearm_skin_10_fixed_joint: type fixed, parent l_forearm, child l_forearm_skin_10, origin xyz=0.0542285210888 0.007546 -0.0321469082866 rpy=-2.94123313406 -0.328304471922 -0.0139662781936
- added joint l_forearm_skin_11_fixed_joint: type fixed, parent l_forearm, child l_forearm_skin_11, origin xyz=0.0542240912024 -0.0112832 -0.0321431259452 rpy=2.93929835957 -0.329101389745 0.0142734891292
- added joint l_forearm_skin_12_fixed_joint: type fixed, parent l_forearm, child l_forearm_skin_12, origin xyz=0.0375994633868 -0.0204556 -0.0340191179961 rpy=2.58303505964 -0.29483050207 0.021326850448
- added joint l_forearm_skin_13_fixed_joint: type fixed, parent l_forearm, child l_forearm_skin_13, origin xyz=0.0228550868405 -0.0112878 -0.0418919009209 rpy=2.94896679198 -0.270583947189 0.00177385006765
- added joint l_forearm_skin_14_fixed_joint: type fixed, parent l_forearm, child l_forearm_skin_14, origin xyz=0.0687703276364 -0.0193999 -0.0230239558511 rpy=2.52462250363 -0.387794511771 0.0912924111683
- added joint l_forearm_skin_15_fixed_joint: type fixed, parent l_forearm, child l_forearm_skin_15, origin xyz=0.0633786419662 -0.0293843 -0.00879405455544 rpy=1.80492769741 -0.289783281916 0.113933739306
- added joint l_forearm_skin_16_fixed_joint: type fixed, parent l_forearm, child l_forearm_skin_16, origin xyz=0.03792482187 -0.0327268 0.0206369503605 rpy=1.41280007026 -0.25082462139 0.0758652301584
- added joint l_forearm_skin_17_fixed_joint: type fixed, parent l_forearm, child l_forearm_skin_17, origin xyz=0.0543170548821 -0.0299646 0.0303291240179 rpy=1.27223716205 -0.23059304703 0.109637225219
- added joint l_forearm_skin_19_fixed_joint: type fixed, parent l_forearm, child l_forearm_skin_19, origin xyz=0.0381266107138 0.029054 0.020690605393 rpy=-1.41560888703 -0.252569290226 -0.0644404747027
- added joint l_forearm_skin_1_fixed_joint: type fixed, parent l_forearm, child l_forearm_skin_1, origin xyz=0.0333728935826 -0.0310662 -0.0198456867711 rpy=1.86694023278 -0.274442533764 0.0421228737473
- added joint l_forearm_skin_22_fixed_joint: type fixed, parent l_forearm, child l_forearm_skin_22, origin xyz=0.0544173950421 0.026483 0.0306037516609 rpy=-1.2658242728 -0.234328151379 -0.0937094738802
- added joint l_forearm_skin_24_fixed_joint: type fixed, parent l_forearm, child l_forearm_skin_24, origin xyz=0.0700345319564 0.007477 0.050069108714 rpy=-0.23489327644 -0.0388172993982 -0.0548291989999
- added joint l_forearm_skin_25_fixed_joint: type fixed, parent l_forearm, child l_forearm_skin_25, origin xyz=0.0535999216295 0.015984 0.0454698125045 rpy=-0.564295527715 -0.136980272197 -0.0819608256656
- added joint l_forearm_skin_28_fixed_joint: type fixed, parent l_forearm, child l_forearm_skin_28, origin xyz=0.0535859272148 -0.0196522 0.045352037397 rpy=0.579311106949 -0.133994306778 0.0867597858312
- added joint l_forearm_skin_29_fixed_joint: type fixed, parent l_forearm, child l_forearm_skin_29, origin xyz=0.0700355805031 -0.0111936 0.0500111036233 rpy=0.248630982209 -0.0383136556786 0.0583026624266
- added joint l_forearm_skin_2_fixed_joint: type fixed, parent l_forearm, child l_forearm_skin_2, origin xyz=0.0146988929852 -0.0335184 -0.0160117338371 rpy=1.72847287019 -0.264015219116 0.0142600467197
- added joint l_forearm_skin_3_fixed_joint: type fixed, parent l_forearm, child l_forearm_skin_3, origin xyz=0.045567293622 0.028651 -0.00633000929351 rpy=-1.69487280859 -0.269757727104 -0.061995217851
- added joint l_forearm_skin_4_fixed_joint: type fixed, parent l_forearm, child l_forearm_skin_4, origin xyz=0.0635326332996 0.025877 -0.00899784258066 rpy=-1.81747870108 -0.287406884885 -0.0998316152826
- added joint l_forearm_skin_5_fixed_joint: type fixed, parent l_forearm, child l_forearm_skin_5, origin xyz=0.0688211941968 0.015709 -0.0231133361791 rpy=-2.5410475806 -0.385627260642 -0.0867227569203
- added joint l_forearm_skin_6_fixed_joint: type fixed, parent l_forearm, child l_forearm_skin_6, origin xyz=0.0333948436255 0.027308 -0.0198325583433 rpy=-1.86628164653 -0.272886336181 -0.0371068033783
- added joint l_forearm_skin_7_fixed_joint: type fixed, parent l_forearm, child l_forearm_skin_7, origin xyz=0.0147224260074 0.029702 -0.0159326482703 rpy=-1.72564640857 -0.263992900722 -0.0143801109253
- added joint l_forearm_skin_8_fixed_joint: type fixed, parent l_forearm, child l_forearm_skin_8, origin xyz=0.0228528628554 0.007546 -0.041885146375 rpy=-2.94801979137 -0.270605090512 -0.00178708074348
- added joint l_forearm_skin_9_fixed_joint: type fixed, parent l_forearm, child l_forearm_skin_9, origin xyz=0.0376032734683 0.016715 -0.0340163371186 rpy=-2.58406517708 -0.2933217196 -0.0203085796276
- added joint l_hand_dh_frame_fixed_joint: type fixed, parent l_hand, child l_hand_dh_frame, origin xyz=0.0576542978428 -0.0055568 0.0136938323083 rpy=-1.57079632679 -0.261799319827 0
- added joint l_wrist_pitch: type revolute, parent l_forearm, child l_wrist_1, origin xyz=0.103427563179 7.00000000002e-06 0.0254874807467 rpy=0 0 0, axis 0.258818979447 0.0 -0.965925843882, limit lower=-1.3962634016 upper=0.436332312999 effort=50000 velocity=50000
- added joint l_wrist_prosup: type revolute, parent l_elbow_1, child l_forearm, origin xyz=0.0384624299027 0.0339999 -0.00522316819403 rpy=0 0 0, axis 0.965925843882 2.22044604925e-16 0.258818979447, limit lower=-1.0471975512 upper=1.0471975512 effort=50000 velocity=50000
- added joint l_wrist_yaw: type revolute, parent l_wrist_1, child l_hand, origin xyz=-0.000634106499644 -0.0194999 0.00236651831751 rpy=0 0 0, axis -2.22044604925e-16 1.0 0.0, limit lower=-0.349065850399 upper=0.436332312999 effort=50000 velocity=50000
- added joint r_forearm_dh_frame_fixed_joint: type fixed, parent r_forearm, child r_forearm_dh_frame, origin xyz=-0.102871102373 7.00000000002e-06 0.0275642213111 rpy=-0.261799319827 0 -1.57079632679
- added joint r_forearm_skin_0_fixed_joint: type fixed, parent r_forearm, child r_forearm_skin_0, origin xyz=-0.0454493286618 0.030077 -0.00628656037901 rpy=1.69181522292 -0.271026744341 -3.06880438227
- added joint r_forearm_skin_10_fixed_joint: type fixed, parent r_forearm, child r_forearm_skin_10, origin xyz=-0.0542285210888 -0.0097861 -0.0321469082866 rpy=-2.94123313406 -0.328304471922 3.1276263754
- added joint r_forearm_skin_11_fixed_joint: type fixed, parent r_forearm, child r_forearm_skin_11, origin xyz=-0.0542240912024 0.009043 -0.0321431259452 rpy=2.93929835957 -0.329101389745 -3.12731916446
- added joint r_forearm_skin_12_fixed_joint: type fixed, parent r_forearm, child r_forearm_skin_12, origin xyz=-0.0375994633868 0.018216 -0.0340191179961 rpy=2.58303505964 -0.29483050207 -3.12026580314
- added joint r_forearm_skin_13_fixed_joint: type fixed, parent r_forearm, child r_forearm_skin_13, origin xyz=-0.0228550868405 0.009048 -0.0418919009209 rpy=2.94896679198 -0.270583947189 -3.13981880352
- added joint r_forearm_skin_14_fixed_joint: type fixed, parent r_forearm, child r_forearm_skin_14, origin xyz=-0.0687703276364 0.01716 -0.0230239558511 rpy=2.48044991868 -0.295542566281 -2.91877349139
- added joint r_forearm_skin_15_fixed_joint: type fixed, parent r_forearm, child r_forearm_skin_15, origin xyz=-0.0633786419662 0.027145 -0.00879405455544 rpy=1.80492769741 -0.289783281916 -3.02765891428
- added joint r_forearm_skin_16_fixed_joint: type fixed, parent r_forearm, child r_forearm_skin_16, origin xyz=-0.03792482187 0.030487 0.0206369503605 rpy=1.41280007026 -0.25082462139 -3.06572742343
- added joint r_forearm_skin_17_fixed_joint: type fixed, parent r_forearm, child r_forearm_skin_17, origin xyz=-0.0543170548821 0.027725 0.0303291240179 rpy=1.27223716205 -0.23059304703 -3.03195542837
- added joint r_forearm_skin_19_fixed_joint: type fixed, parent r_forearm, child r_forearm_skin_19, origin xyz=-0.0381266107138 -0.0312941 0.020690605393 rpy=-1.41560888703 -0.252569290226 3.07715217889
- added joint r_forearm_skin_1_fixed_joint: type fixed, parent r_forearm, child r_forearm_skin_1, origin xyz=-0.0333728935826 0.028826 -0.0198456867711 rpy=1.86694023278 -0.274442533764 -3.09946977984
- added joint r_forearm_skin_22_fixed_joint: type fixed, parent r_forearm, child r_forearm_skin_22, origin xyz=-0.0544173950421 -0.0287223 0.0306037516609 rpy=-1.2658242728 -0.234328151379 3.04788317971
- added joint r_forearm_skin_24_fixed_joint: type fixed, parent r_forearm, child r_forearm_skin_24, origin xyz=-0.0700345319564 -0.0097164 0.050069108714 rpy=-0.23489327644 -0.0388172993982 3.08676345459
- added joint r_forearm_skin_25_fixed_joint: type fixed, parent r_forearm, child r_forearm_skin_25, origin xyz=-0.0535999216295 -0.0182238 0.0454698125045 rpy=-0.564295527715 -0.136980272197 3.05963182792
- added joint r_forearm_skin_28_fixed_joint: type fixed, parent r_forearm, child r_forearm_skin_28, origin xyz=-0.0535859272148 0.017412 0.045352037397 rpy=0.59077064408 -0.0531607226063 3.10597081167
- added joint r_forearm_skin_29_fixed_joint: type fixed, parent r_forearm, child r_forearm_skin_29, origin xyz=-0.0700355805031 0.008954 0.0500111036233 rpy=0.248630982209 -0.0383136556786 -3.08328999116
- added joint r_forearm_skin_2_fixed_joint: type fixed, parent r_forearm, child r_forearm_skin_2, origin xyz=-0.0146988929852 0.031279 -0.0160117338371 rpy=1.72847287019 -0.264015219116 -3.12733260687
- added joint r_forearm_skin_3_fixed_joint: type fixed, parent r_forearm, child r_forearm_skin_3, origin xyz=-0.045567293622 -0.030891 -0.00633000929351 rpy=-1.69487280859 -0.269757727104 3.07959743574
- added joint r_forearm_skin_4_fixed_joint: type fixed, parent r_forearm, child r_forearm_skin_4, origin xyz=-0.0635326332996 -0.0281163 -0.00899784258066 rpy=-1.80734960194 -0.0393131796327 2.97997643632
- added joint r_forearm_skin_5_fixed_joint: type fixed, parent r_forearm, child r_forearm_skin_5, origin xyz=-0.0688211941968 -0.0179483 -0.0231133361791 rpy=-2.5410475806 -0.385627260642 3.05486989667
- added joint r_forearm_skin_6_fixed_joint: type fixed, parent r_forearm, child r_forearm_skin_6, origin xyz=-0.0333948436255 -0.0295479 -0.0198325583433 rpy=-1.86628164653 -0.272886336181 3.10448585021
- added joint r_forearm_skin_7_fixed_joint: type fixed, parent r_forearm, child r_forearm_skin_7, origin xyz=-0.0147224260074 -0.0319422 -0.0159326482703 rpy=-1.72564640857 -0.263992900722 3.12721254266
- added joint r_forearm_skin_8_fixed_joint: type fixed, parent r_forearm, child r_forearm_skin_8, origin xyz=-0.0228528628554 -0.0097862 -0.041885146375 rpy=-2.94801979137 -0.270605090512 3.13980557285
- added joint r_forearm_skin_9_fixed_joint: type fixed, parent r_forearm, child r_forearm_skin_9, origin xyz=-0.0376032734683 -0.018955 -0.0340163371186 rpy=-2.58406517708 -0.2933217196 3.12128407396
- added joint r_hand_dh_frame_fixed_joint: type fixed, parent r_hand, child r_hand_dh_frame, origin xyz=-0.0576542978428 -0.0055568 0.0136938323083 rpy=-1.57079632679 -0.261799319827 3.14159265359
- added joint r_wrist_pitch: type revolute, parent r_forearm, child r_wrist_1, origin xyz=-0.103505208873 7.00000000002e-06 0.0251977029936 rpy=0 0 0, axis 0.258818979447 0.0 0.965925843882, limit lower=-1.3962634016 upper=0.436332312999 effort=50000 velocity=50000
- added joint r_wrist_prosup: type revolute, parent r_elbow_1, child r_forearm, origin xyz=-0.0384624299027 0.0224999 -0.00522316819403 rpy=0 0 0, axis -0.965925843882 2.22044604925e-16 0.258818979447, limit lower=-1.0471975512 upper=1.0471975512 effort=50000 velocity=50000
- added joint r_wrist_yaw: type revolute, parent r_wrist_1, child r_hand, origin xyz=0.000634106499644 -0.0194999 0.00236651831751 rpy=0 0 0, axis 2.22044604925e-16 1.0 0.0, limit lower=-0.349065850399 upper=0.436332312999 effort=50000 velocity=50000
- joint chest_ems_acc_eb1_fixed_joint: origin xyz=0.0647855001907 0.064043 -0.064709 rpy=3.1415169123 -0.261799309122 0.000292641880255 -> xyz=0.0647855001907 0.064043 -0.0647091 rpy=3.1415169123 -0.261799309122 0.000292641880255
- joint chest_ems_acc_eb4_fixed_joint: origin xyz=-0.0621620998093 0.088063 -0.0529886 rpy=-3.14159050476 -0.261799319819 3.14158433987 -> xyz=-0.0621620998093 0.088063 -0.0529887 rpy=-3.14159050476 -0.261799319819 3.14158433987
- joint chest_ems_gyro_eb1_fixed_joint: origin xyz=0.0692016001907 0.064548 -0.0635257 rpy=3.1415169123 -0.261799309122 0.000292641880255 -> xyz=0.0692016001907 0.064548 -0.0635258 rpy=3.1415169123 -0.261799309122 0.000292641880255
- joint chest_ems_gyro_eb2_fixed_joint: origin xyz=0.0160371001907 0.087559 -0.0653478 rpy=3.14159050104 0.261799319819 3.14158433678 -> xyz=0.0160371001907 0.087559 -0.0653479 rpy=3.14159050104 0.261799319819 3.14158433678
- joint chest_ems_gyro_eb4_fixed_joint: origin xyz=-0.0665783998093 0.087559 -0.0518053 rpy=-3.14159050476 -0.261799319819 3.14158433987 -> xyz=-0.0665783998093 0.087559 -0.0518054 rpy=-3.14159050476 -0.261799319819 3.14158433987
- joint chest_mtb_acc_0b10_fixed_joint: origin xyz=0.0594286001907 -0.0018543 0.0457982 rpy=-0.875168153475 0.116362025479 -1.65561807505 -> xyz=0.0594286001907 -0.0018543 0.0457981 rpy=-0.875168153475 0.116362025479 -1.65561807505
- joint chest_mtb_acc_0b7_fixed_joint: origin xyz=-0.0607539998093 -0.0017836 0.0442342 rpy=0.875167771492 0.116363734392 -1.48597350247 -> xyz=-0.0607539998093 -0.0017836 0.0442341 rpy=0.875167771492 0.116363734392 -1.48597350247
- joint l_ankle_pitch: origin xyz=0.0592832 -0.201 0 rpy=0 0 0 -> xyz=0.0406034 -0.2005 0 rpy=0 0 0
- joint l_ankle_roll: origin xyz=-0.0355 0 0.04808755 rpy=0 0 0 -> xyz=-0.0270179 0 0.04808755 rpy=0 0 0
- joint l_forearm_mtb_acc_1b7_fixed_joint: origin xyz=0.114369314675 0.0285169 -0.0165299963729 rpy=0.26179949998 0.000370413042328 -1.57033448496 -> xyz=0.0768727847342 -0.005483 -0.0110479126068 rpy=0.26179949998 0.000370413042328 -1.57033448496; parent l_elbow_1 -> l_forearm
- joint l_forearm_mtb_acc_1b8_fixed_joint: origin xyz=0.088920691578 0.015972 0.035268688442 rpy=-0.661143946092 0.147825248461 -3.04952253889 -> xyz=0.0514241740607 -0.0180279 0.0407507258436 rpy=-0.661143946092 0.147825248461 -3.04952253889; parent l_elbow_1 -> l_forearm
- joint l_forearm_mtb_acc_1b9_fixed_joint: origin xyz=0.0595957174403 0.0596569 -0.0205995080872 rpy=1.76682134218 0.261099829847 3.08752548202 -> xyz=0.0220991874996 0.025657 -0.0151174243212 rpy=1.76682134218 0.261099829847 3.08752548202; parent l_elbow_1 -> l_forearm
- joint l_knee: axis -1.0 -0.0 -0.0 -> -1.0 0.0 0.0; origin xyz=-0.0237832 -0.145625 0 rpy=0 0 0 -> xyz=-0.0135855 -0.145625 0 rpy=0 0 0
- joint l_lower_leg_ems_acc_eb7_fixed_joint: origin xyz=0.0350978 -0.092765 0.04351373 rpy=0 -0.218166543341 1.57079632679 -> xyz=0.0249001 -0.092765 0.04351373 rpy=0 -0.218166543341 1.57079632679
- joint l_lower_leg_ems_gyro_eb7_fixed_joint: origin xyz=0.0356017 -0.088301 0.044503292 rpy=0 -0.218166543341 1.57079632679 -> xyz=0.025404 -0.088301 0.044503292 rpy=0 -0.218166543341 1.57079632679
- joint l_lower_leg_mtb_acc_10b10_fixed_joint: origin xyz=0.030989 -0.011037 0.05238133 rpy=-1.32645042367 0 1.57079632679 -> xyz=0.0563295 -0.043468 0.0259151 rpy=1.30899714594 -0.000112159802878 1.57082638021
- joint l_lower_leg_mtb_acc_10b11_fixed_joint: origin xyz=-0.0179355 -0.092958 0.0184593 rpy=-1.3089971472 -2.54317885716e-05 1.57078951235 -> xyz=-0.0281332 -0.092958 0.0184593 rpy=-1.3089971472 -2.54317885716e-05 1.57078951235
- joint l_lower_leg_mtb_acc_10b8_fixed_joint: origin xyz=0.0099841 -0.004318 0.0544518 rpy=-0.349065638045 3.97141037841e-05 1.57090544048 -> xyz=0.0307696 -0.004318 0.05313347 rpy=0.24434616607 0 1.57079632679
- joint l_lower_leg_mtb_acc_10b9_fixed_joint: origin xyz=0.0665272 -0.043468 0.0259151 rpy=1.30899714594 -0.000112159802878 1.57082638021 -> xyz=-0.0002136 -0.004318 0.0544518 rpy=-0.349065638045 3.97141037841e-05 1.57090544048
- joint l_shoulder_pitch: origin xyz=0.120016000191 0.0928 0.0079694 rpy=0 0 0 -> xyz=0.120016000191 0.0928 0.0079693 rpy=0 0 0
- joint l_shoulder_roll: origin xyz=-0.013671 0 0.0085203 rpy=0.270597317916 0.252680177542 -1.50155688559 -> xyz=-0.013671 0 0.0085204 rpy=0.270597317916 0.252680177542 -1.50155688559
- joint l_shoulder_yaw: origin xyz=0.0253143218312 1.37518334151e-07 -0.00540052326137 rpy=-0.252689546175 -0.0085186183214 -0.067039889142 -> xyz=0.0253143468312 1.11636438205e-07 -0.00540061656265 rpy=-0.252689546175 -0.0085186183214 -0.067039889142
- joint l_upper_arm_mtb_acc_1b12_fixed_joint: origin xyz=-0.0412195 -0.029588 0.0049921 rpy=-1.57079718993 -1.57078381225 2.68257161162 -> xyz=-0.0412194 -0.029588 0.0049921 rpy=-1.57079718993 -1.57078381225 2.68257161162
- joint l_upper_arm_mtb_acc_1b13_fixed_joint: origin xyz=0.010592657 -0.028351 -0.0086914 rpy=-1.57079632657 0.000214520362042 -2.47803674451 -> xyz=0.010592709 -0.028351 -0.0086914 rpy=-1.57079632657 0.000214520362042 -2.47803674451
- joint l_upper_leg_mtb_acc_10b2_fixed_joint: origin xyz=0.0083839 0.039452 0.05335544 rpy=0.837758036965 -8.62912869137e-05 1.57087402394 -> xyz=0.0083839 0.039452 0.05335544 rpy=0.261799318135 -3.00531353284e-05 1.57090848663
- joint neck_roll: origin xyz=0.0142999998093 0.0095 0.02080001 rpy=0 0 0 -> xyz=0.0142999998093 0.0095 0.02079997 rpy=0 0 0
- joint neck_yaw: origin xyz=0 -0.022344 -0.02080001 rpy=0 0 0 -> xyz=0 -0.022344 -0.02079997 rpy=0 0 0
- joint r_ankle_pitch: origin xyz=-0.0593039 -0.201 0 rpy=0 0 0 -> xyz=-0.0188325 -0.2005 0 rpy=0 0 0
- joint r_ankle_roll: axis -0.0 -0.0 -1.0 -> 0.0 0.0 -1.0; origin xyz=0.0355 0 -0.0185 rpy=0 0 0 -> xyz=0.0285 0 -0.0185 rpy=0 0 0
- joint r_forearm_mtb_acc_2b7_fixed_joint: origin xyz=-0.114369314675 0.0279969 -0.0165299963729 rpy=0.26179949998 0.000370413042328 1.57125816863 -> xyz=-0.0768727847342 0.005497 -0.0110479126068 rpy=0.26179949998 0.000370413042328 1.57125816863; parent r_elbow_1 -> r_forearm
- joint r_forearm_mtb_acc_2b8_fixed_joint: origin xyz=-0.0891879954459 0.0037515 0.034800424042 rpy=0.661159832193 0.147746087249 -0.0919671195152 -> xyz=-0.0514186150796 0.015786 0.0407521537277 rpy=-0.661143946092 0.147825248461 0.092070114703; parent r_elbow_1 -> r_forearm
- joint r_forearm_mtb_acc_2b9_fixed_joint: origin xyz=-0.0591345256166 0.0504239 -0.0187311091679 rpy=-1.76682626732 0.261191225646 0.054048344372 -> xyz=-0.0216379956759 0.027924 -0.0132490254018 rpy=-1.76682626732 0.261191225646 0.054048344372; parent r_elbow_1 -> r_forearm
- joint r_hip_pitch: axis -1.0 -0.0 -0.0 -> -1.0 0.0 0.0
- joint r_hip_roll: axis -0.0 -0.0 -1.0 -> 0.0 0.0 -1.0
- joint r_knee: origin xyz=0.0238039 -0.145625 0 rpy=0 0 0 -> xyz=-0.0096675 -0.145625 0 rpy=0 0 0
- joint r_lower_leg_ems_acc_eb9_fixed_joint: origin xyz=-0.0099643 -0.092765 0.04351373 rpy=0 -0.218166543341 1.57079632679 -> xyz=0.0235071 -0.092765 0.04351373 rpy=0 -0.218166543341 1.57079632679
- joint r_lower_leg_ems_gyro_eb9_fixed_joint: origin xyz=-0.0094604 -0.088301 0.044503292 rpy=0 -0.218166543341 1.57079632679 -> xyz=0.024011 -0.088301 0.044503292 rpy=0 -0.218166543341 1.57079632679
- joint r_lower_leg_mtb_acc_11b10_fixed_joint: origin xyz=-0.0389997 -0.004318 0.05362922 rpy=-0.244346164565 2.80911040962e-05 1.57090899435 -> xyz=-0.0325465 -0.043468 0.0278945 rpy=-1.30899714732 0 1.57079632679
- joint r_lower_leg_mtb_acc_11b11_fixed_joint: origin xyz=0.0184451 -0.092958 0.0164801 rpy=1.30899714594 -0.000112159802878 1.57082638021 -> xyz=0.0519165 -0.092958 0.0164801 rpy=1.30899714594 -0.000112159802878 1.57082638021
- joint r_lower_leg_mtb_acc_11b8_fixed_joint: origin xyz=-0.008081 -0.004318 0.0537517 rpy=0.349065638046 -3.97141043948e-05 1.57090544048 -> xyz=-0.0055283 -0.004318 0.05362922 rpy=-0.244346164565 2.80911040962e-05 1.57090899435
- joint r_lower_leg_mtb_acc_11b9_fixed_joint: origin xyz=-0.0660179 -0.043468 0.0278945 rpy=-1.30899714732 0 1.57079632679 -> xyz=0.0253904 -0.004318 0.0537517 rpy=0.349065638045 -3.97141037841e-05 1.57090544048
- joint r_shoulder_pitch: origin xyz=-0.120015999809 0.0928 0.0079694 rpy=0 -0.523598883792 3.14159265359 -> xyz=-0.120015999809 0.0928 0.0079693 rpy=0 -0.523598883792 3.14159265359
- joint r_upper_arm_mtb_acc_2b10_fixed_joint: origin xyz=-0.0412195 0.029588 0.0295279 rpy=1.57079546365 1.57078381225 -2.68257161164 -> xyz=-0.0412194 0.029588 0.0295279 rpy=1.57079546365 1.57078381225 -2.68257161164
- joint r_upper_arm_mtb_acc_2b12_fixed_joint: origin xyz=-0.0430555 0.028681 0.0049922 rpy=-1.11177442168 -1.57079632679 0 -> xyz=-0.0430554 0.028681 0.0049922 rpy=-1.11177442168 -1.57079632679 0
- joint r_upper_arm_mtb_acc_2b13_fixed_joint: origin xyz=0.010593184 0.02835 -0.010738 rpy=1.57079632702 -0.000214520362041 2.47803674451 -> xyz=0.010593237 0.02835 -0.010738 rpy=1.57079632702 -0.000214520362041 2.47803674451
- joint r_upper_leg_mtb_acc_11b2_fixed_joint: origin xyz=-0.0064065 0.039256 0.0539467 rpy=-0.837758053858 -0.000342790749344 1.57087401652 -> xyz=-0.0064065 0.039256 0.0539467 rpy=-0.261799341927 -0.000399050135154 1.57090848318
- joint torso_roll: origin xyz=0.0270462998093 0.032 -0.0576906 rpy=0 0 0 -> xyz=0.0270462998093 0.032 -0.0573446 rpy=0 0 0
- joint torso_yaw: origin xyz=0 0.05 0.0631871 rpy=0 0 0 -> xyz=0 0.05 0.0628421 rpy=0 0 0
