Commit message: [iCubGenova02] Fix sign of r_wrist_prosup axis

File: app/robots/iCubGenova02/model.urdf (robot description, URDF)
Before this commit: robot ICUB_2-5_BB_SIM_MODEL, 163 links, 162 joints
Joints:
- joint r_wrist_prosup: axis -0.965925843882 2.22044604925e-16 0.258818979447 -> 0.965925843882 -2.22044604925e-16 -0.258818979447

Commit message: added contact frames on icub legs

File: app/robots/iCubGenova02/model.urdf (robot description, URDF)
Before this commit: robot ICUB_2-5_BB_SIM_MODEL, 163 links, 162 joints
Links:
- added link l_upper_leg_contact
- added link r_upper_leg_contact
Joints:
- added joint l_upper_leg_contact_fixed_joint: type fixed, parent l_upper_leg, child l_upper_leg_contact, origin xyz=-0.0003 0.0146 -0.0512571 rpy=0 0 1.57079632679
- added joint r_upper_leg_contact_fixed_joint: type fixed, parent r_upper_leg, child r_upper_leg_contact, origin xyz=0.0003 0.0146 -0.0512571 rpy=0 0 1.57079632679

Commit message: Update model.urdf

File: app/robots/iCubGenova02/model.urdf (robot description, URDF)
Before this commit: robot ICUB_2-5_BB_SIM_MODEL, 165 links, 164 joints
Joints:
- joint l_upper_leg_contact_fixed_joint: origin xyz=-0.0003 0.0146 -0.0512571 rpy=0 0 1.57079632679 -> xyz=-0.0003 0.0146 -0.0512571 rpy=0 0 -1.57079632679
- joint r_upper_leg_contact_fixed_joint: origin xyz=0.0003 0.0146 -0.0512571 rpy=0 0 1.57079632679 -> xyz=0.0003 0.0146 -0.0512571 rpy=0 0 -1.57079632679
