Commit message: [iCubDarmstad01] New model for iCub Darmstad 01, based on iCubGenova02
The main difference was in the chest link, beacuse iCub Darmstadt does not have
the backpack. This difference was evaluted to be approximatly 2 kilograms,
and the com of the chest was moved to be consistent with the COM of the old
model of iCubGenova01 .

File: app/robots/iCubDarmstadt01/model.urdf (robot description, URDF)
Before this commit: robot iCub, 56 links, 55 joints
Links:
- removed link chest_skin_frame
- removed link codyco_balancing_world
- removed link l_forearm
- removed link l_forearm_dh_frame
- removed link l_gripper
- removed link l_hand
- removed link l_hand_dh_frame
- removed link l_upper_arm_dh_frame
- removed link l_wrist_1
- removed link r_forearm
- removed link r_forearm_dh_frame
- removed link r_gripper
- removed link r_hand
- removed link r_hand_dh_frame
- removed link r_upper_arm_dh_frame
- removed link r_wrist_1
- removed link torso
- added link chest_ems_acc_eb1
- added link chest_ems_acc_eb2
- added link chest_ems_acc_eb3
- added link chest_ems_acc_eb4
- added link chest_ems_gyro_eb1
- added link chest_ems_gyro_eb2
- added link chest_ems_gyro_eb3
- added link chest_ems_gyro_eb4
- added link chest_mtb_acc_0b10
- added link chest_mtb_acc_0b7
- added link chest_mtb_acc_0b8
- added link chest_mtb_acc_0b9
- added link l_foot_mtb_acc_10b12
- added link l_foot_mtb_acc_10b13
- added link l_forearm_mtb_acc_1b7
- added link l_forearm_mtb_acc_1b8
- added link l_forearm_mtb_acc_1b9
- added link l_lower_leg_ems_acc_eb7
- added link l_lower_leg_ems_gyro_eb7
- added link l_lower_leg_mtb_acc_10b10
- added link l_lower_leg_mtb_acc_10b11
- added link l_lower_leg_mtb_acc_10b8
- added link l_lower_leg_mtb_acc_10b9
- added link l_upper_arm_mtb_acc_1b10
- added link l_upper_arm_mtb_acc_1b11
- added link l_upper_arm_mtb_acc_1b12
- added link l_upper_arm_mtb_acc_1b13
- added link l_upper_leg_ems_acc_eb10
- added link l_upper_leg_ems_acc_eb6
- added link l_upper_leg_ems_gyro_eb10
- added link l_upper_leg_ems_gyro_eb6
- added link l_upper_leg_mtb_acc_10b1
- added link l_upper_leg_mtb_acc_10b2
- added link l_upper_leg_mtb_acc_10b3
- added link l_upper_leg_mtb_acc_10b4
- added link l_upper_leg_mtb_acc_10b5
- added link l_upper_leg_mtb_acc_10b6
- added link l_upper_leg_mtb_acc_10b7
- added link r_foot_mtb_acc_11b12
- added link r_foot_mtb_acc_11b13
- added link r_forearm_mtb_acc_2b7
- added link r_forearm_mtb_acc_2b8
- added link r_forearm_mtb_acc_2b9
- added link r_lower_leg_ems_acc_eb9
- added link r_lower_leg_ems_gyro_eb9
- added link r_lower_leg_mtb_acc_11b10
- added link r_lower_leg_mtb_acc_11b11
- added link r_lower_leg_mtb_acc_11b8
- added link r_lower_leg_mtb_acc_11b9
- added link r_upper_arm_mtb_acc_2b10
- added link r_upper_arm_mtb_acc_2b11
- added link r_upper_arm_mtb_acc_2b12
- added link r_upper_arm_mtb_acc_2b13
- added link r_upper_leg_ems_acc_eb11
- added link r_upper_leg_ems_acc_eb8
- added link r_upper_leg_ems_gyro_eb11
- added link r_upper_leg_ems_gyro_eb8
- added link r_upper_leg_mtb_acc_11b1
- added link r_upper_leg_mtb_acc_11b2
- added link r_upper_leg_mtb_acc_11b3
- added link r_upper_leg_mtb_acc_11b4
- added link r_upper_leg_mtb_acc_11b5
- added link r_upper_leg_mtb_acc_11b6
- added link r_upper_leg_mtb_acc_11b7
- added link root_link_ems_acc_eb5
- added link root_link_ems_gyro_eb5
- link chest: mass 4.81 -> 5.638; geometry collision mesh filename=model://iCubGenova02/meshes/dae/bb_chest.dae scale=0.001 0.001 0.001; visual mesh filename=model://iCubGenova02/meshes/dae/bb_chest.dae scale=0.001 0.001 0.001
- link head: mass 3 -> 1.50691; geometry collision mesh filename=model://iCubGenova02/meshes/dae/head.dae scale=0.001 0.001 0.001; visual mesh filename=model://iCubGenova02/meshes/dae/head.dae scale=0.001 0.001 0.001
- link imu_frame: mass 0 -> None
- link l_ankle_1: mass 0.643 -> 0.6798; geometry collision mesh filename=model://iCubGenova02/meshes/dae/l_ankle_1.dae scale=0.001 0.001 0.001; visual mesh filename=model://iCubGenova02/meshes/dae/l_ankle_1.dae scale=0.001 0.001 0.001
- link l_ankle_2: mass 0.2675 -> 0.267485; geometry collision mesh filename=model://iCubGenova02/meshes/dae/l_ankle_2.dae scale=0.001 0.001 0.001; visual mesh filename=model://iCubGenova02/meshes/dae/l_ankle_2.dae scale=0.001 0.001 0.001
- link l_elbow_1: mass 0.074 -> 1.17718; geometry collision mesh filename=model://iCubGenova02/meshes/dae/l_elbow_1.dae scale=0.001 0.001 0.001; visual mesh filename=model://iCubGenova02/meshes/dae/l_elbow_1.dae scale=0.001 0.001 0.001
- link l_foot: mass 0.5935 -> 0.382372; geometry collision mesh filename=model://iCubGenova02/meshes/dae/l_foot.dae scale=0.001 0.001 0.001; visual mesh filename=model://iCubGenova02/meshes/dae/l_foot.dae scale=0.001 0.001 0.001
- link l_foot_dh_frame: mass 0 -> None
- link l_hip_1: mass 0.695 -> 0.915608; geometry collision mesh filename=model://iCubGenova02/meshes/dae/l_hip_1.dae scale=0.001 0.001 0.001; visual mesh filename=model://iCubGenova02/meshes/dae/l_hip_1.dae scale=0.001 0.001 0.001
- link l_hip_2: mass 0.982 -> 0.421161; geometry collision mesh filename=model://iCubGenova02/meshes/dae/l_hip_2.dae scale=0.001 0.001 0.001; visual mesh filename=model://iCubGenova02/meshes/dae/l_hip_2.dae scale=0.001 0.001 0.001
- link l_hip_3: mass 0 -> 0.126212; geometry collision mesh filename=model://iCubGenova02/meshes/dae/l_hip_3.dae scale=0.001 0.001 0.001; visual mesh filename=model://iCubGenova02/meshes/dae/l_hip_3.dae scale=0.001 0.001 0.001
- link l_lower_leg: mass 2.032 -> 1.4724; geometry collision mesh filename=model://iCubGenova02/meshes/dae/l_lower_leg.dae scale=0.001 0.001 0.001; visual mesh filename=model://iCubGenova02/meshes/dae/l_lower_leg.dae scale=0.001 0.001 0.001
- link l_shoulder_1: mass 0.189 -> 0.114882; geometry collision mesh filename=model://iCubGenova02/meshes/dae/l_shoulder_1.dae scale=0.001 0.001 0.001; visual mesh filename=model://iCubGenova02/meshes/dae/l_shoulder_1.dae scale=0.001 0.001 0.001
- link l_shoulder_2: mass 0.179 -> 0.239074; geometry collision mesh filename=model://iCubGenova02/meshes/dae/l_shoulder_2.dae scale=0.001 0.001 0.001; visual mesh filename=model://iCubGenova02/meshes/dae/l_shoulder_2.dae scale=0.001 0.001 0.001
- link l_shoulder_3: mass 0.156157 -> 0.35913; geometry collision mesh filename=model://iCubGenova02/meshes/dae/l_shoulder_3.dae scale=0.001 0.001 0.001; visual mesh filename=model://iCubGenova02/meshes/dae/l_shoulder_3.dae scale=0.001 0.001 0.001
- link l_sole: mass 0 -> None
- link l_upper_arm: mass 0.727843 -> 0.746799; geometry collision mesh filename=model://iCubGenova02/meshes/dae/l_upper_arm.dae scale=0.001 0.001 0.001; visual mesh filename=model://iCubGenova02/meshes/dae/l_upper_arm.dae scale=0.001 0.001 0.001
- link l_upper_leg: mass 1.522 -> 1.8084; geometry collision mesh filename=model://iCubGenova02/meshes/dae/l_upper_leg.dae scale=0.001 0.001 0.001; visual mesh filename=model://iCubGenova02/meshes/dae/l_upper_leg.dae scale=0.001 0.001 0.001
- link neck_1: mass 0 -> 0.125793; geometry collision mesh filename=model://iCubGenova02/meshes/dae/neck_1.dae scale=0.001 0.001 0.001; visual mesh filename=model://iCubGenova02/meshes/dae/neck_1.dae scale=0.001 0.001 0.001
- link neck_2: mass 0 -> 0.177087; geometry collision mesh filename=model://iCubGenova02/meshes/dae/neck_2.dae scale=0.001 0.001 0.001; visual mesh filename=model://iCubGenova02/meshes/dae/neck_2.dae scale=0.001 0.001 0.001
- link r_ankle_1: mass 0.643 -> 0.6803; geometry collision mesh filename=model://iCubGenova02/meshes/dae/r_ankle_1.dae scale=0.001 0.001 0.001; visual mesh filename=model://iCubGenova02/meshes/dae/r_ankle_1.dae scale=0.001 0.001 0.001
- link r_ankle_2: mass 0.2675 -> 0.267485; geometry collision mesh filename=model://iCubGenova02/meshes/dae/r_ankle_2.dae scale=0.001 0.001 0.001; visual mesh filename=model://iCubGenova02/meshes/dae/r_ankle_2.dae scale=0.001 0.001 0.001
- link r_elbow_1: mass 0.074 -> 1.17637; geometry collision mesh filename=model://iCubGenova02/meshes/dae/r_elbow_1.dae scale=0.001 0.001 0.001; visual mesh filename=model://iCubGenova02/meshes/dae/r_elbow_1.dae scale=0.001 0.001 0.001
- link r_foot: mass 0.5935 -> 0.38227; geometry collision mesh filename=model://iCubGenova02/meshes/dae/r_foot.dae scale=0.001 0.001 0.001; visual mesh filename=model://iCubGenova02/meshes/dae/r_foot.dae scale=0.001 0.001 0.001
- link r_foot_dh_frame: mass 0 -> None
- link r_hip_1: mass 0.695 -> 0.920354; geometry collision mesh filename=model://iCubGenova02/meshes/dae/r_hip_1.dae scale=0.001 0.001 0.001; visual mesh filename=model://iCubGenova02/meshes/dae/r_hip_1.dae scale=0.001 0.001 0.001
- link r_hip_2: mass 0.982 -> 0.4194; geometry collision mesh filename=model://iCubGenova02/meshes/dae/r_hip_2.dae scale=0.001 0.001 0.001; visual mesh filename=model://iCubGenova02/meshes/dae/r_hip_2.dae scale=0.001 0.001 0.001
- link r_hip_3: mass 0 -> 0.126212; geometry collision mesh filename=model://iCubGenova02/meshes/dae/r_hip_3.dae scale=0.001 0.001 0.001; visual mesh filename=model://iCubGenova02/meshes/dae/r_hip_3.dae scale=0.001 0.001 0.001
- link r_lower_leg: mass 2.032 -> 1.472; geometry collision mesh filename=model://iCubGenova02/meshes/dae/r_lower_leg.dae scale=0.001 0.001 0.001; visual mesh filename=model://iCubGenova02/meshes/dae/r_lower_leg.dae scale=0.001 0.001 0.001
- link r_shoulder_1: mass 0.189 -> 0.114862; geometry collision mesh filename=model://iCubGenova02/meshes/dae/r_shoulder_1.dae scale=0.001 0.001 0.001; visual mesh filename=model://iCubGenova02/meshes/dae/r_shoulder_1.dae scale=0.001 0.001 0.001
- link r_shoulder_2: mass 0.179 -> 0.238162; geometry collision mesh filename=model://iCubGenova02/meshes/dae/r_shoulder_2.dae scale=0.001 0.001 0.001; visual mesh filename=model://iCubGenova02/meshes/dae/r_shoulder_2.dae scale=0.001 0.001 0.001
- link r_shoulder_3: mass 0.155 -> 0.35913; geometry collision mesh filename=model://iCubGenova02/meshes/dae/r_shoulder_3.dae scale=0.001 0.001 0.001; visual mesh filename=model://iCubGenova02/meshes/dae/r_shoulder_3.dae scale=0.001 0.001 0.001
- link r_sole: mass 0 -> None
- link r_upper_arm: mass 0.729 -> 0.745104; geometry collision mesh filename=model://iCubGenova02/meshes/dae/r_upper_arm.dae scale=0.001 0.001 0.001; visual mesh filename=model://iCubGenova02/meshes/dae/r_upper_arm.dae scale=0.001 0.001 0.001
- link r_upper_leg: mass 1.522 -> 1.8035; geometry collision mesh filename=model://iCubGenova02/meshes/dae/r_upper_leg.dae scale=0.001 0.001 0.001; visual mesh filename=model://iCubGenova02/meshes/dae/r_upper_leg.dae scale=0.001 0.001 0.001
- link root_link: mass 4.72 -> 5.09143; geometry collision mesh filename=model://iCubGenova02/meshes/dae/root.dae scale=0.001 0.001 0.001; visual mesh filename=model://iCubGenova02/meshes/dae/root.dae scale=0.001 0.001 0.001
- link torso_1: mass 0 -> 0.67144; geometry collision mesh filename=model://iCubGenova02/meshes/dae/torso_1.dae scale=0.001 0.001 0.001; visual mesh filename=model://iCubGenova02/meshes/dae/torso_1.dae scale=0.001 0.001 0.001
- link torso_2: mass 0 -> 0.428161; geometry collision mesh filename=model://iCubGenova02/meshes/dae/torso_2.dae scale=0.001 0.001 0.001; visual mesh filename=model://iCubGenova02/meshes/dae/torso_2.dae scale=0.001 0.001 0.001
Joints:
- removed joint chest_skin_frame_fixed_joint
- removed joint codyco_balancing_world_fixed_joint
- removed joint l_forearm_dh_frame_fixed_joint
- removed joint l_gripper_joint
- removed joint l_hand_dh_frame_fixed_joint
- removed joint l_upper_arm_dh_frame_fixed_joint
- removed joint l_wrist_pitch
- removed joint l_wrist_prosup
- removed joint l_wrist_yaw
- removed joint r_forearm_dh_frame_fixed_joint
- removed joint r_gripper_joint
- removed joint r_hand_dh_frame_fixed_joint
- removed joint r_upper_arm_dh_frame_fixed_joint
- removed joint r_wrist_pitch
- removed joint r_wrist_prosup
- removed joint r_wrist_yaw
- removed joint torso_joint
- added joint chest_ems_acc_eb1_fixed_joint: type fixed, parent chest, child chest_ems_acc_eb1, origin xyz=0.0647855001907 0.064043 -0.064709 rpy=3.1415169123 -0.261799309122 0.000292641880255
- added joint chest_ems_acc_eb2_fixed_joint: type fixed, parent chest, child chest_ems_acc_eb2, origin xyz=0.0204533001907 0.088063 -0.0641645 rpy=3.14159050104 0.261799319819 3.14158433678
- added joint chest_ems_acc_eb3_fixed_joint: type fixed, parent chest, child chest_ems_acc_eb3, origin xyz=-0.0230587998093 0.064019 -0.0758985 rpy=3.14110916203 0.261100516471 -0.000309071462555
- added joint chest_ems_acc_eb4_fixed_joint: type fixed, parent chest, child chest_ems_acc_eb4, origin xyz=-0.0621620998093 0.088063 -0.0529886 rpy=-3.14159050476 -0.261799319819 3.14158433987
- added joint chest_ems_gyro_eb1_fixed_joint: type fixed, parent chest, child chest_ems_gyro_eb1, origin xyz=0.0692016001907 0.064548 -0.0635257 rpy=3.1415169123 -0.261799309122 0.000292641880255
- added joint chest_ems_gyro_eb2_fixed_joint: type fixed, parent chest, child chest_ems_gyro_eb2, origin xyz=0.0160371001907 0.087559 -0.0653478 rpy=3.14159050104 0.261799319819 3.14158433678
- added joint chest_ems_gyro_eb3_fixed_joint: type fixed, parent chest, child chest_ems_gyro_eb3, origin xyz=-0.0186416998093 0.064521 -0.0770785 rpy=3.14110916203 0.261100516471 -0.000309071462555
- added joint chest_ems_gyro_eb4_fixed_joint: type fixed, parent chest, child chest_ems_gyro_eb4, origin xyz=-0.0665783998093 0.087559 -0.0518053 rpy=-3.14159050476 -0.261799319819 3.14158433987
- added joint chest_mtb_acc_0b10_fixed_joint: type fixed, parent chest, child chest_mtb_acc_0b10, origin xyz=0.0594286001907 -0.0018543 0.0457982 rpy=-0.875168153475 0.116362025479 -1.65561807505
- added joint chest_mtb_acc_0b7_fixed_joint: type fixed, parent chest, child chest_mtb_acc_0b7, origin xyz=-0.0607539998093 -0.0017836 0.0442342 rpy=0.875167771492 0.116363734392 -1.48597350247
- added joint chest_mtb_acc_0b8_fixed_joint: type fixed, parent chest, child chest_mtb_acc_0b8, origin xyz=-0.0457046998093 -0.001846 0.0567427 rpy=0.500960084689 0.107313688983 -1.4778325291
- added joint chest_mtb_acc_0b9_fixed_joint: type fixed, parent chest, child chest_mtb_acc_0b9, origin xyz=0.0439036001907 -0.0017841 0.0577221 rpy=-0.500959928973 0.107315404248 -1.66376017469
- added joint l_foot_mtb_acc_10b12_fixed_joint: type fixed, parent l_foot, child l_foot_mtb_acc_10b12, origin xyz=0.1055224 0.0008072 -0.001215 rpy=0 0 1.57079632679
- added joint l_foot_mtb_acc_10b13_fixed_joint: type fixed, parent l_foot, child l_foot_mtb_acc_10b13, origin xyz=0.0805224 0.0118072 -0.001215 rpy=0 0 1.57079632679
- added joint l_forearm_mtb_acc_1b7_fixed_joint: type fixed, parent l_elbow_1, child l_forearm_mtb_acc_1b7, origin xyz=0.114369314675 0.0285169 -0.0165299963729 rpy=0.26179949998 0.000370413042328 -1.57033448496
- added joint l_forearm_mtb_acc_1b8_fixed_joint: type fixed, parent l_elbow_1, child l_forearm_mtb_acc_1b8, origin xyz=0.088920691578 0.015972 0.035268688442 rpy=-0.661143946092 0.147825248461 -3.04952253889
- added joint l_forearm_mtb_acc_1b9_fixed_joint: type fixed, parent l_elbow_1, child l_forearm_mtb_acc_1b9, origin xyz=0.0595957174403 0.0596569 -0.0205995080872 rpy=1.76682134218 0.261099829847 3.08752548202
- added joint l_lower_leg_ems_acc_eb7_fixed_joint: type fixed, parent l_lower_leg, child l_lower_leg_ems_acc_eb7, origin xyz=0.0350978 -0.092765 0.04351373 rpy=0 -0.218166543341 1.57079632679
- added joint l_lower_leg_ems_gyro_eb7_fixed_joint: type fixed, parent l_lower_leg, child l_lower_leg_ems_gyro_eb7, origin xyz=0.0356017 -0.088301 0.044503292 rpy=0 -0.218166543341 1.57079632679
- added joint l_lower_leg_mtb_acc_10b10_fixed_joint: type fixed, parent l_lower_leg, child l_lower_leg_mtb_acc_10b10, origin xyz=0.030989 -0.011037 0.05238133 rpy=-1.32645042367 0 1.57079632679
- added joint l_lower_leg_mtb_acc_10b11_fixed_joint: type fixed, parent l_lower_leg, child l_lower_leg_mtb_acc_10b11, origin xyz=-0.0179355 -0.092958 0.0184593 rpy=-1.3089971472 -2.54317885716e-05 1.57078951235
- added joint l_lower_leg_mtb_acc_10b8_fixed_joint: type fixed, parent l_lower_leg, child l_lower_leg_mtb_acc_10b8, origin xyz=0.0099841 -0.004318 0.0544518 rpy=-0.349065638045 3.97141037841e-05 1.57090544048
- added joint l_lower_leg_mtb_acc_10b9_fixed_joint: type fixed, parent l_lower_leg, child l_lower_leg_mtb_acc_10b9, origin xyz=0.0665272 -0.043468 0.0259151 rpy=1.30899714594 -0.000112159802878 1.57082638021
- added joint l_upper_arm_mtb_acc_1b10_fixed_joint: type fixed, parent l_upper_arm, child l_upper_arm_mtb_acc_1b10, origin xyz=-0.0430554 -0.028681 0.0295279 rpy=-1.57079650664 -1.57050350741 2.68257092837
- added joint l_upper_arm_mtb_acc_1b11_fixed_joint: type fixed, parent l_upper_arm, child l_upper_arm_mtb_acc_1b11, origin xyz=-0.0412181 -0.029589 0.0760604 rpy=-1.57079650664 -1.57050350741 2.68257092837
- added joint l_upper_arm_mtb_acc_1b12_fixed_joint: type fixed, parent l_upper_arm, child l_upper_arm_mtb_acc_1b12, origin xyz=-0.0412195 -0.029588 0.0049921 rpy=-1.57079718993 -1.57078381225 2.68257161162
- added joint l_upper_arm_mtb_acc_1b13_fixed_joint: type fixed, parent l_upper_arm, child l_upper_arm_mtb_acc_1b13, origin xyz=0.010592657 -0.028351 -0.0086914 rpy=-1.57079632657 0.000214520362042 -2.47803674451
- added joint l_upper_leg_ems_acc_eb10_fixed_joint: type fixed, parent l_upper_leg, child l_upper_leg_ems_acc_eb10, origin xyz=0.040407 -0.040027 -0.0125751 rpy=1.57079632679 0 1.57079632679
- added joint l_upper_leg_ems_acc_eb6_fixed_joint: type fixed, parent l_upper_leg, child l_upper_leg_ems_acc_eb6, origin xyz=-0.0404072 -0.083207 -0.0125771 rpy=1.57079632679 0 -1.57079632679
- added joint l_upper_leg_ems_gyro_eb10_fixed_joint: type fixed, parent l_upper_leg, child l_upper_leg_ems_gyro_eb10, origin xyz=0.040407 -0.035455 -0.013079 rpy=1.57079632679 0 1.57079632679
- added joint l_upper_leg_ems_gyro_eb6_fixed_joint: type fixed, parent l_upper_leg, child l_upper_leg_ems_gyro_eb6, origin xyz=-0.0404072 -0.087779 -0.013081 rpy=1.57079632679 0 -1.57079632679
- added joint l_upper_leg_mtb_acc_10b1_fixed_joint: type fixed, parent l_upper_leg, child l_upper_leg_mtb_acc_10b1, origin xyz=0.031565 0.049332 0.04200163 rpy=0.837758036961 -8.62912829653e-05 1.57087402394
- added joint l_upper_leg_mtb_acc_10b2_fixed_joint: type fixed, parent l_upper_leg, child l_upper_leg_mtb_acc_10b2, origin xyz=0.0083839 0.039452 0.05335544 rpy=0.837758036965 -8.62912869137e-05 1.57087402394
- added joint l_upper_leg_mtb_acc_10b3_fixed_joint: type fixed, parent l_upper_leg, child l_upper_leg_mtb_acc_10b3, origin xyz=0.0150706 0.004382 0.053785 rpy=0 0 1.57079632679
- added joint l_upper_leg_mtb_acc_10b4_fixed_joint: type fixed, parent l_upper_leg, child l_upper_leg_mtb_acc_10b4, origin xyz=-0.0144294 0.004382 0.053785 rpy=0 0 1.57079632679
- added joint l_upper_leg_mtb_acc_10b5_fixed_joint: type fixed, parent l_upper_leg, child l_upper_leg_mtb_acc_10b5, origin xyz=-0.0414999 -0.004658 0.03412949 rpy=-1.18682376254 0 1.57079632679
- added joint l_upper_leg_mtb_acc_10b6_fixed_joint: type fixed, parent l_upper_leg, child l_upper_leg_mtb_acc_10b6, origin xyz=0.0178086 -0.026212 -0.043785 rpy=3.14159265359 0 -1.57091243005
- added joint l_upper_leg_mtb_acc_10b7_fixed_joint: type fixed, parent l_upper_leg, child l_upper_leg_mtb_acc_10b7, origin xyz=-0.0141918 -0.026211 -0.043785 rpy=3.14159265359 0 -1.5709453147
- added joint r_foot_mtb_acc_11b12_fixed_joint: type fixed, parent r_foot, child r_foot_mtb_acc_11b12, origin xyz=0.1034744 -0.000807 -0.001215 rpy=0 0 -1.57079632679
- added joint r_foot_mtb_acc_11b13_fixed_joint: type fixed, parent r_foot, child r_foot_mtb_acc_11b13, origin xyz=0.0784744 -0.0118072 -0.001215 rpy=0 0 -1.57079632679
- added joint r_forearm_mtb_acc_2b7_fixed_joint: type fixed, parent r_elbow_1, child r_forearm_mtb_acc_2b7, origin xyz=-0.114369314675 0.0279969 -0.0165299963729 rpy=0.26179949998 0.000370413042328 1.57125816863
- added joint r_forearm_mtb_acc_2b8_fixed_joint: type fixed, parent r_elbow_1, child r_forearm_mtb_acc_2b8, origin xyz=-0.0891879954459 0.0037515 0.034800424042 rpy=0.661159832193 0.147746087249 -0.0919671195152
- added joint r_forearm_mtb_acc_2b9_fixed_joint: type fixed, parent r_elbow_1, child r_forearm_mtb_acc_2b9, origin xyz=-0.0591345256166 0.0504239 -0.0187311091679 rpy=-1.76682626732 0.261191225646 0.054048344372
- added joint r_lower_leg_ems_acc_eb9_fixed_joint: type fixed, parent r_lower_leg, child r_lower_leg_ems_acc_eb9, origin xyz=-0.0099643 -0.092765 0.04351373 rpy=0 -0.218166543341 1.57079632679
- added joint r_lower_leg_ems_gyro_eb9_fixed_joint: type fixed, parent r_lower_leg, child r_lower_leg_ems_gyro_eb9, origin xyz=-0.0094604 -0.088301 0.044503292 rpy=0 -0.218166543341 1.57079632679
- added joint r_lower_leg_mtb_acc_11b10_fixed_joint: type fixed, parent r_lower_leg, child r_lower_leg_mtb_acc_11b10, origin xyz=-0.0389997 -0.004318 0.05362922 rpy=-0.244346164565 2.80911040962e-05 1.57090899435
- added joint r_lower_leg_mtb_acc_11b11_fixed_joint: type fixed, parent r_lower_leg, child r_lower_leg_mtb_acc_11b11, origin xyz=0.0184451 -0.092958 0.0164801 rpy=1.30899714594 -0.000112159802878 1.57082638021
- added joint r_lower_leg_mtb_acc_11b8_fixed_joint: type fixed, parent r_lower_leg, child r_lower_leg_mtb_acc_11b8, origin xyz=-0.008081 -0.004318 0.0537517 rpy=0.349065638046 -3.97141043948e-05 1.57090544048
- added joint r_lower_leg_mtb_acc_11b9_fixed_joint: type fixed, parent r_lower_leg, child r_lower_leg_mtb_acc_11b9, origin xyz=-0.0660179 -0.043468 0.0278945 rpy=-1.30899714732 0 1.57079632679
- added joint r_upper_arm_mtb_acc_2b10_fixed_joint: type fixed, parent r_upper_arm, child r_upper_arm_mtb_acc_2b10, origin xyz=-0.0412195 0.029588 0.0295279 rpy=1.57079546365 1.57078381225 -2.68257161164
- added joint r_upper_arm_mtb_acc_2b11_fixed_joint: type fixed, parent r_upper_arm, child r_upper_arm_mtb_acc_2b11, origin xyz=-0.0430568 0.02868 0.0760604 rpy=-1.57079614696 -1.57050350741 0.459021725219
- added joint r_upper_arm_mtb_acc_2b12_fixed_joint: type fixed, parent r_upper_arm, child r_upper_arm_mtb_acc_2b12, origin xyz=-0.0430555 0.028681 0.0049922 rpy=-1.11177442168 -1.57079632679 0
- added joint r_upper_arm_mtb_acc_2b13_fixed_joint: type fixed, parent r_upper_arm, child r_upper_arm_mtb_acc_2b13, origin xyz=0.010593184 0.02835 -0.010738 rpy=1.57079632702 -0.000214520362041 2.47803674451
- added joint r_upper_leg_ems_acc_eb11_fixed_joint: type fixed, parent r_upper_leg, child r_upper_leg_ems_acc_eb11, origin xyz=-0.040407 -0.083207 -0.0125771 rpy=1.57079632679 0 -1.57079632679
- added joint r_upper_leg_ems_acc_eb8_fixed_joint: type fixed, parent r_upper_leg, child r_upper_leg_ems_acc_eb8, origin xyz=0.0404072 -0.040027 -0.0125751 rpy=1.57079632679 0 -1.57079632679
- added joint r_upper_leg_ems_gyro_eb11_fixed_joint: type fixed, parent r_upper_leg, child r_upper_leg_ems_gyro_eb11, origin xyz=-0.040407 -0.087779 -0.013081 rpy=1.57079632679 0 -1.57079632679
- added joint r_upper_leg_ems_gyro_eb8_fixed_joint: type fixed, parent r_upper_leg, child r_upper_leg_ems_gyro_eb8, origin xyz=0.0404072 -0.035455 -0.013079 rpy=1.57079632679 0 -1.57079632679
- added joint r_upper_leg_mtb_acc_11b1_fixed_joint: type fixed, parent r_upper_leg, child r_upper_leg_mtb_acc_11b1, origin xyz=-0.030195 0.04914 0.043588612 rpy=-0.837758053858 -0.000342790749344 1.57087401652
- added joint r_upper_leg_mtb_acc_11b2_fixed_joint: type fixed, parent r_upper_leg, child r_upper_leg_mtb_acc_11b2, origin xyz=-0.0064065 0.039256 0.0539467 rpy=-0.837758053858 -0.000342790749344 1.57087401652
- added joint r_upper_leg_mtb_acc_11b3_fixed_joint: type fixed, parent r_upper_leg, child r_upper_leg_mtb_acc_11b3, origin xyz=-0.0130214 0.004186 0.0538313 rpy=0 -0.000429089990594 1.57091244355
- added joint r_upper_leg_mtb_acc_11b4_fixed_joint: type fixed, parent r_upper_leg, child r_upper_leg_mtb_acc_11b4, origin xyz=0.0422675 -0.004845 0.0322719 rpy=1.18682375086 -0.000536853726193 1.57083983106
- added joint r_upper_leg_mtb_acc_11b5_fixed_joint: type fixed, parent r_upper_leg, child r_upper_leg_mtb_acc_11b5, origin xyz=0.0164786 0.004186 0.0538313 rpy=0 -0.000429089990594 1.57091244355
- added joint r_upper_leg_mtb_acc_11b6_fixed_joint: type fixed, parent r_upper_leg, child r_upper_leg_mtb_acc_11b6, origin xyz=-0.0157594 -0.026365 -0.0437518 rpy=3.14159265359 0.000429089993416 -1.57079632679
- added joint r_upper_leg_mtb_acc_11b7_fixed_joint: type fixed, parent r_upper_leg, child r_upper_leg_mtb_acc_11b7, origin xyz=0.0162386 -0.026366 -0.0437518 rpy=3.14159260377 0.000429089990404 -1.57091243007
- added joint root_link_ems_acc_eb5_fixed_joint: type fixed, parent root_link, child root_link_ems_acc_eb5, origin xyz=0.0493308 -0.0125771 -0.115691 rpy=3.14159265359 1.29154404503 3.14159265359
- added joint root_link_ems_gyro_eb5_fixed_joint: type fixed, parent root_link, child root_link_ems_gyro_eb5, origin xyz=0.0493308 -0.0125771 -0.115691 rpy=3.14159265359 1.29154404503 3.14159265359
- joint imu_frame_fixed_joint: axis 0 0 0 -> (none); origin xyz=0.0185 -0.1108 0.0066 rpy=1.5708 -0 0 -> xyz=0.00950000019074 0.133444 0.0093 rpy=-1.57079632679 1.57079632679 0
- joint l_ankle_pitch: axis 0 -1 6.12323e-17 -> 1.0 0.0 0.0; limit lower=-0.733038 upper=0.366519 effort=24 velocity=100 -> lower=-0.349065850399 upper=0.523598775598 effort=50000 velocity=50000; origin xyz=-0.2005 0 0 rpy=-1.5708 0 0 -> xyz=0.0592832 -0.201 0 rpy=0 0 0
- joint l_ankle_roll: axis 1 0 0 -> 0.0 0.0 1.0; limit lower=-0.418879 upper=0.418879 effort=11 velocity=100 -> lower=-0.349065850399 upper=0.349065850399 effort=50000 velocity=50000; origin xyz=0 0 0 rpy=0 -1.5708 0 -> xyz=-0.0355 0 0.04808755 rpy=0 0 0
- joint l_arm_ft_sensor: axis 0 0 0 -> (none); origin xyz=0.015 9.36797e-18 0.068 rpy=0 -0 0 -> xyz=0.0509301432452 0 0.0291758294659 rpy=0 -1.30899700697 3.14159265359
- joint l_elbow: axis 0 1 6.12323e-17 -> 2.22044604925e-16 -1.0 0.0; limit lower=0.0959931 upper=1.85005 effort=20 velocity=100 -> lower=0.261799387799 upper=1.85004900711 effort=50000 velocity=50000; origin xyz=0 0 0.08428 rpy=-6.12323e-17 0 0 -> xyz=0 0.0339999 0.07926 rpy=0 -1.30899700697 -3.14159265359
- joint l_foot_dh_frame_fixed_joint: origin xyz=0 0 0.004 rpy=0 1.5708 0 -> xyz=0.0 0 0.004 rpy=0 1.5708 0
- joint l_foot_ft_sensor: axis 0 0 0 -> (none); origin xyz=-0.0035 0 0.0645 rpy=0 -0 0 -> xyz=0 -0.0603 -0.05158755 rpy=1.57079632679 -1.57079632679 0
- joint l_hip_pitch: axis 0 -1 6.12323e-17 -> -1.0 0.0 0.0; limit lower=-0.767945 upper=2.30383 effort=84 velocity=100 -> lower=-0.523598775598 upper=1.4835298642 effort=50000 velocity=50000; origin xyz=0 -0.0681 -0.1199 rpy=-3.14159 1.5708 -2.77556e-17 -> xyz=0.0064515 -0.0223861 -0.119913 rpy=1.57079632679 0 -1.57079632679
- joint l_hip_roll: axis 1 0 -6.12323e-17 -> 0.0 0.0 1.0; limit lower=-2.07694 upper=0.296706 effort=84 velocity=100 -> lower=0.0 upper=1.57079632679 effort=50000 velocity=50000; origin xyz=0 0 0 rpy=3.14159 -1.5708 -2.77556e-17 -> xyz=0.0477139 0 -0.02554 rpy=0 0 0
- joint l_hip_yaw: axis 0 1 6.12323e-17 -> 0.0 1.0 0.0; limit lower=-1.37881 upper=1.37881 effort=40 velocity=100 -> lower=-1.2217304764 upper=1.2217304764 effort=50000 velocity=50000; origin xyz=0 -1.68519e-34 -0.0665 rpy=-1.5708 -6.16298e-33 -6.12323e-17 -> xyz=0 0 0.0146 rpy=-1.57079632679 0 -1.57079632679
- joint l_knee: axis 0 1.22465e-16 -1 -> -1.0 -0.0 -0.0; limit lower=-2.18166 upper=0.401426 effort=30 velocity=100 -> lower=-1.74532925199 upper=0.0 effort=50000 velocity=50000; origin xyz=-0.0009175 -0.234545 -1.43617e-17 rpy=3.14159 -1.2326e-32 1.5708 -> xyz=-0.0237832 -0.145625 0 rpy=0 0 0
- joint l_leg_ft_sensor: axis 0 0 0 -> (none); origin xyz=0 0 0.0665 rpy=0 -0 0 -> xyz=0 -0.0743 0.0246825 rpy=1.57079632679 -1.57079632679 0
- joint l_shoulder_pitch: axis 0 -1 5.55112e-17 -> 0.965926 0.0 0.258819; limit lower=-1.65806 upper=0.0872665 effort=84 velocity=100 -> lower=-1.66678943565 upper=0.174532925199 effort=50000 velocity=50000; origin xyz=0.00525 0.1433 -0.11026 rpy=1.309 5.55112e-17 1.5708 -> xyz=0.120016000191 0.0928 0.0079694 rpy=0 0 0
- joint l_shoulder_roll: axis 0 1 6.12323e-17 -> -0.258819 2.77555756156e-17 0.965926; limit lower=0 upper=2.80649 effort=84 velocity=100 -> lower=0.0 upper=2.80648943721 effort=50000 velocity=50000; origin xyz=0 0 0 rpy=1.5708 -0 -1.5708 -> xyz=-0.013671 0 0.0085203 rpy=0.270597317916 0.252680177542 -1.50155688559
- joint l_shoulder_yaw: axis 0 6.12323e-17 1 -> 0.965925843882 2.22044604925e-16 0.258818979447; limit lower=-0.645772 upper=1.74533 effort=34 velocity=100 -> lower=-0.645771823238 upper=1.3962634016 effort=50000 velocity=50000; origin xyz=4.33681e-19 1.73472e-18 0 rpy=6.12323e-17 -0 1.309 -> xyz=0.0253143218312 1.37518334151e-07 -0.00540052326137 rpy=-0.252689546175 -0.0085186183214 -0.067039889142
- joint l_sole_fixed_joint: axis 0 0 0 -> (none); origin xyz=-8.67362e-19 -1.38778e-17 0.004 rpy=3.14159 -0 0 -> xyz=0.0035 0 0.004 rpy=-3.14159265359 0 0
- joint neck_pitch: axis 0 1 6.12323e-17 -> -1.0 0.0 0.0; limit lower=-0.698132 upper=0.523599 effort=20 velocity=100 -> lower=-0.698131700798 upper=0.383972435439 effort=50000 velocity=50000; origin xyz=0.00231 0.1933 -1.18362e-17 rpy=1.5708 -0 1.5708 -> xyz=-0.0142999998093 0.172797 0.0053118 rpy=0 0 0
- joint neck_roll: axis 0 -1 6.12323e-17 -> 0.0 0.0 1.0; limit lower=-1.22173 upper=1.0472 effort=20 velocity=100 -> lower=-0.349065850399 upper=0.349065850399 effort=50000 velocity=50000; origin xyz=0.0095 0 0 rpy=-1.5708 -0 -1.5708 -> xyz=0.0142999998093 0.0095 0.02080001 rpy=0 0 0
- joint neck_yaw: axis 0 -1 6.12323e-17 -> 0.0 1.0 0.0; limit lower=-0.959931 upper=0.959931 effort=20 velocity=100 -> lower=-0.872664625997 upper=0.872664625997 effort=50000 velocity=50000; origin xyz=-5.77779e-34 0 0 rpy=-1.5708 -0 1.5708 -> xyz=0 -0.022344 -0.02080001 rpy=0 0 0
- joint r_ankle_pitch: axis 0 1 6.12323e-17 -> 1.0 0.0 0.0; limit lower=-0.733038 upper=0.366519 effort=24 velocity=100 -> lower=-0.349065850399 upper=0.523598775598 effort=50000 velocity=50000; origin xyz=-0.2005 0 0 rpy=1.5708 -0 0 -> xyz=-0.0593039 -0.201 0 rpy=0 0 0
- joint r_ankle_roll: axis -1 1.22465e-16 0 -> -0.0 -0.0 -1.0; limit lower=-0.418879 upper=0.418879 effort=11 velocity=100 -> lower=-0.349065850399 upper=0.349065850399 effort=50000 velocity=50000; origin xyz=0 0 0 rpy=0.504019 1.5708 -2.63757 -> xyz=0.0355 0 -0.0185 rpy=0 0 0
- joint r_arm_ft_sensor: axis 0 0 0 -> (none); origin xyz=0.015 -8.93429e-18 0.068 rpy=0 -0 0 -> xyz=-0.0508973017665 0 0.0291670296206 rpy=0 -1.30899700697 0
- joint r_elbow: axis 0 1 6.12323e-17 -> 2.22044604925e-16 1.0 0.0; limit lower=0.0959931 upper=1.85005 effort=20 velocity=100 -> lower=0.261799387799 upper=1.85004900711 effort=50000 velocity=50000; origin xyz=0 0 0.08428 rpy=3.14159 -0 3.14159 -> xyz=0 -0.0224999 0.07926 rpy=0 1.30899700697 0
- joint r_foot_dh_frame_fixed_joint: origin xyz=0 0 0.004 rpy=0 1.5708 0 -> xyz=0.0 0 0.004 rpy=0 1.5708 0
- joint r_foot_ft_sensor: axis 0 0 0 -> (none); origin xyz=-0.0035 4.28626e-19 0.0645 rpy=0 -0 0 -> xyz=0 -0.0603 0.015 rpy=1.57079632679 -1.57079632679 0
- joint r_hip_pitch: axis 0 1 6.12323e-17 -> -1.0 -0.0 -0.0; limit lower=-0.767945 upper=2.30383 effort=84 velocity=100 -> lower=-0.523598775598 upper=1.4835298642 effort=50000 velocity=50000; origin xyz=0 0.0681 -0.1199 rpy=-2.77556e-17 1.5708 2.77556e-17 -> xyz=0.0064515 0.0233655 -0.119913 rpy=1.57079632679 0 -1.57079632679
- joint r_hip_roll: axis -1 0 6.12323e-17 -> -0.0 -0.0 -1.0; limit lower=-2.07694 upper=0.296706 effort=84 velocity=100 -> lower=0.0 upper=1.57079632679 effort=50000 velocity=50000; origin xyz=0 0 0 rpy=2.77556e-17 1.5708 -2.77556e-17 -> xyz=-0.0467345 0 -0.0263447 rpy=0 0 0
- joint r_hip_yaw: axis 0 -1 6.12323e-17 -> 0.0 -1.0 0.0; limit lower=-1.37881 upper=1.37881 effort=40 velocity=100 -> lower=-1.2217304764 upper=1.2217304764 effort=50000 velocity=50000; origin xyz=0 1.68519e-34 -0.0665 rpy=-1.5708 -6.16298e-33 6.12323e-17 -> xyz=0 0 0.0146 rpy=-1.57079632679 0 -1.57079632679
- joint r_knee: axis 0 1.22465e-16 -1 -> -1.0 0.0 0.0; limit lower=-2.18166 upper=0.401426 effort=30 velocity=100 -> lower=-1.74532925199 upper=0.0 effort=50000 velocity=50000; origin xyz=-0.0009175 -0.234545 1.43617e-17 rpy=3.14159 -1.2326e-32 1.5708 -> xyz=0.0238039 -0.145625 0 rpy=0 0 0
- joint r_leg_ft_sensor: axis 0 0 0 -> (none); origin xyz=0 0 0.0665 rpy=0 -0 0 -> xyz=0 -0.0743 0.0254872 rpy=1.57079632679 -1.57079632679 0
- joint r_shoulder_pitch: axis 0 1 5.55112e-17 -> -0.965925926173 0.0 0.258819275525; limit lower=-1.65806 upper=0.0872665 effort=84 velocity=100 -> lower=-1.66678943565 upper=0.174532925199 effort=50000 velocity=50000; origin xyz=0.00525 0.1433 0.11026 rpy=-1.309 -0 1.5708 -> xyz=-0.120015999809 0.0928 0.0079694 rpy=0 -0.523598883792 3.14159265359
- joint r_shoulder_roll: axis 0 -1 6.12323e-17 -> -0.258819 -2.77555756156e-17 -0.965926; limit lower=0 upper=2.80649 effort=84 velocity=100 -> lower=0.0 upper=2.80648943721 effort=50000 velocity=50000; origin xyz=0 0 0 rpy=-1.5708 -0 -1.5708 -> xyz=-0.00758046573227 0 0.0142102463639 rpy=-0.270597611583 -0.252680154648 -1.50155680035
- joint r_shoulder_yaw: axis 0 6.12323e-17 -1 -> 0.965925843882 -2.22044604925e-16 -0.258818979447; limit lower=-0.645772 upper=1.74533 effort=34 velocity=100 -> lower=-0.645771823238 upper=1.3962634016 effort=50000 velocity=50000; origin xyz=-4.33681e-19 0 0 rpy=3.14159 -0 1.309 -> xyz=-0.0253460713232 2.32750427306e-07 -0.00538764806457 rpy=-0.252689546175 0.0085186183214 0.067039889142
- joint r_sole_fixed_joint: axis 0 0 0 -> (none); origin xyz=-8.67362e-19 1.38778e-17 0.004 rpy=3.14159 -0 0 -> xyz=0.0035 0 0.004 rpy=-3.14159265359 0 0
- joint torso_pitch: axis 0 1 6.12323e-17 -> 1.0 0.0 0.0; limit lower=-0.383972 upper=1.46608 effort=36 velocity=100 -> lower=-0.349065850399 upper=1.2217304764 effort=50000 velocity=50000; origin xyz=0 0 0 rpy=-2.77556e-17 -1.5708 3.14159 -> xyz=0 0.0270463 0 rpy=1.57079632679 0 -1.57079632679
- joint torso_roll: axis 0 1 6.12323e-17 -> 0.0 0.0 -1.0; limit lower=-0.680678 upper=0.680678 effort=80 velocity=100 -> lower=-0.523598775598 upper=0.523598775598 effort=50000 velocity=50000; origin xyz=0.032 -2.67276e-51 0 rpy=1.5708 -0 -1.5708 -> xyz=0.0270462998093 0.032 -0.0576906 rpy=0 0 0
- joint torso_yaw: axis 0 -1 6.12323e-17 -> 0.0 -1.0 0.0; limit lower=-1.02974 upper=1.02974 effort=80 velocity=100 -> lower=-0.872664625997 upper=0.872664625997 effort=50000 velocity=50000; origin xyz=-7.46298e-34 -0.0055 0 rpy=-1.5708 -0 -1.5708 -> xyz=0 0.05 0.0631871 rpy=0 0 0
