Commit message: new model for walkman

File: app/robots/bigman/bigman_torqueBalancing.urdf (robot description, URDF)
Before this commit: robot bigman, 85 links, 84 joints
Links:
- added link crane_ft
- link DWL: mass 1.44965471 -> 1.635; geometry collision mesh filename=package://bigman_urdf/meshes/walkman/simple/TorsoRoll.STL scale=0.001 0.001 0.001; visual mesh filename=package://bigman_urdf/meshes/walkman/TorsoRoll.STL scale=0.001 0.001 0.001
- link DWS: mass 5.28825567 -> 6.7983647; geometry collision mesh filename=package://bigman_urdf/meshes/walkman/simple/TorsoYawPitch.S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 scale=0.001 0.001 0.001; visual mesh filename=package://bigman_urdf/meshes/walkman/TorsoYawPitch.STL scale=0.001 0.001 0.001
- link DWYTorso: mass 26 -> 9.475; geometry collision mesh filename=package://bigman_urdf/meshes/walkman/simple/NewChest.STL scale=0.001 0.001 0.001; visual mesh filename=package://bigman_urdf/meshes/walkman/NewChest.STL scale=0.001 0.001 0.001
- link LElb: mass 8.6765385e-01 -> 0.8898872; geometry collision mesh filename=package://bigman_urdf/meshes/walkman/simple/Elbow.STL scale=0.001 -0.001 0.001; visual mesh filename=package://bigman_urdf/meshes/walkman/Elbow.STL scale=0.001 -0.001 0.001
- link LFoot: mass 3.42638110 -> 2.58; geometry collision box size=0.32 0.16 0.015; visual mesh filename=package://bigman_urdf/meshes/walkman/NewFoot.STL scale=0.001 -0.001 0.001
- link LFootmot: mass 3.2844159 -> 3.125; geometry collision mesh filename=package://bigman_urdf/meshes/walkman/simple/AnklePitch.STL scale=0.001 -0.001 0.001; visual mesh filename=package://bigman_urdf/meshes/walkman/AnklePitch.STL scale=0.001 -0.001 0.001
- link LForearm: mass 2.2127686 -> 2.17; geometry collision mesh filename=package://bigman_urdf/meshes/walkman/simple/Forearm.STL scale=0.001 -0.001 0.001; visual mesh filename=package://bigman_urdf/meshes/walkman/Forearm.STL scale=0.001 -0.001 0.001
- link LHipMot: mass 3.7958197 -> 4.2423495; geometry collision mesh filename=package://bigman_urdf/meshes/walkman/simple/HipRoll.STL scale=0.001 -0.001 0.001; visual mesh filename=package://bigman_urdf/meshes/walkman/HipRoll.STL scale=0.001 -0.001 0.001
- link LLowLeg: mass 5.6495309 -> 6.82012; geometry collision mesh filename=package://bigman_urdf/meshes/walkman/simple/KneePitchCalf.S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 scale=0.001 -0.001 0.001; visual mesh filename=package://bigman_urdf/meshes/walkman/KneePitchCalf.STL scale=0.001 -0.001 0.001
- link LShp: mass 1.81745527 -> 1.93; geometry collision mesh filename=package://bigman_urdf/meshes/walkman/simple/ShoulderPitch.S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 scale=0.001 -0.001 0.001; visual mesh filename=package://bigman_urdf/meshes/walkman/ShoulderPitch.STL scale=0.001 -0.001 0.001
- link LShr: mass 5.00486460 -> 5.5119737; geometry collision mesh filename=package://bigman_urdf/meshes/walkman/simple/TopUpperArm.STL scale=0.001 -0.001 0.001; visual mesh filename=package://bigman_urdf/meshes/walkman/TopUpperArm.STL scale=0.001 -0.001 0.001
- link LShy: mass 3.20289133 -> 3.1831391; geometry collision mesh filename=package://bigman_urdf/meshes/walkman/simple/BottomUpperArm.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 scale=0.001 -0.001 0.001; visual mesh filename=package://bigman_urdf/meshes/walkman/BottomUpperArm.STL scale=0.001 -0.001 0.001
- link LSoftHandLink: mass 1.2 -> 2.35; geometry collision mesh filename=package://bigman_urdf/meshes/walkman/simple/SoftHandOpen.STL scale=0.001 -0.001 0.001; visual mesh filename=package://bigman_urdf/meshes/walkman/SoftHandOpen.STL scale=0.001 -0.001 0.001
- link LThighLowLeg: mass 5.0950736 -> 5.31976; geometry collision mesh filename=package://bigman_urdf/meshes/walkman/simple/HipPitch.STL scale=0.001 -0.001 0.001; visual mesh filename=package://bigman_urdf/meshes/walkman/HipPitch.STL scale=0.001 -0.001 0.001
- link LThighUpLeg: mass 3.2402068 -> 3.06; geometry collision mesh filename=package://bigman_urdf/meshes/walkman/simple/HipYaw.STL scale=0.001 -0.001 0.001; visual mesh filename=package://bigman_urdf/meshes/walkman/HipYaw.STL scale=0.001 -0.001 0.001
- link LWrMot2: mass 1.2838072 -> 1.195; geometry collision mesh filename=package://bigman_urdf/meshes/walkman/simple/ForearmPitch.STL scale=0.001 -0.001 0.001; visual mesh filename=package://bigman_urdf/meshes/walkman/ForearmPitch.STL scale=0.001 -0.001 0.001
- link LWrMot3: mass 4.2801447e-01 -> 0.175; geometry collision mesh filename=package://bigman_urdf/meshes/walkman/simple/ForearmRoll.STL scale=0.001 -0.001 0.001; visual mesh filename=package://bigman_urdf/meshes/walkman/ForearmRoll.STL scale=0.001 -0.001 0.001
- link NeckPitch: mass 0.623 -> 0.18; geometry collision mesh filename=package://bigman_urdf/meshes/walkman/simple/NeckPitch.STL scale=0.001 0.001 0.001; visual mesh filename=package://bigman_urdf/meshes/walkman/NeckPitch.STL scale=0.001 0.001 0.001
- link NeckYaw: mass 0.35 -> 0.555; geometry collision mesh filename=package://bigman_urdf/meshes/walkman/simple/NeckYaw.STL scale=0.001 0.001 0.001; visual mesh filename=package://bigman_urdf/meshes/walkman/NeckYaw.STL scale=0.001 0.001 0.001
- link RElb: mass 8.6765385e-01 -> 0.8898872; geometry collision mesh filename=package://bigman_urdf/meshes/walkman/simple/Elbow.STL scale=0.001 0.001 0.001; visual mesh filename=package://bigman_urdf/meshes/walkman/Elbow.STL scale=0.001 0.001 0.001
- link RFoot: mass 3.42638110 -> 2.58; geometry collision box size=0.32 0.16 0.015; visual mesh filename=package://bigman_urdf/meshes/walkman/NewFoot.STL scale=0.001 0.001 0.001
- link RFootmot: mass 3.2844159 -> 3.125; geometry collision mesh filename=package://bigman_urdf/meshes/walkman/simple/AnklePitch.STL scale=0.001 0.001 0.001; visual mesh filename=package://bigman_urdf/meshes/walkman/AnklePitch.STL scale=0.001 0.001 0.001
- link RForearm: mass 2.2127686 -> 2.17; geometry collision mesh filename=package://bigman_urdf/meshes/walkman/simple/Forearm.STL scale=0.001 0.001 0.001; visual mesh filename=package://bigman_urdf/meshes/walkman/Forearm.STL scale=0.001 0.001 0.001
- link RHipMot: mass 3.7958197 -> 4.2423495; geometry collision mesh filename=package://bigman_urdf/meshes/walkman/simple/HipRoll.STL scale=0.001 0.001 0.001; visual mesh filename=package://bigman_urdf/meshes/walkman/HipRoll.STL scale=0.001 0.001 0.001
- link RLowLeg: mass 5.6495309 -> 6.82012; geometry collision mesh filename=package://bigman_urdf/meshes/walkman/simple/KneePitchCalf.S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 scale=0.001 0.001 0.001; visual mesh filename=package://bigman_urdf/meshes/walkman/KneePitchCalf.STL scale=0.001 0.001 0.001
- link RShp: mass 1.81745527 -> 1.93; geometry collision mesh filename=package://bigman_urdf/meshes/walkman/simple/ShoulderPitch.S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 scale=0.001 0.001 0.001; visual mesh filename=package://bigman_urdf/meshes/walkman/ShoulderPitch.STL scale=0.001 0.001 0.001
- link RShr: mass 5.00486460 -> 5.5119737; geometry collision mesh filename=package://bigman_urdf/meshes/walkman/simple/TopUpperArm.STL scale=0.001 0.001 0.001; visual mesh filename=package://bigman_urdf/meshes/walkman/TopUpperArm.STL scale=0.001 0.001 0.001
- link RShy: mass 3.20289133 -> 3.1831391; geometry collision mesh filename=package://bigman_urdf/meshes/walkman/simple/BottomUpperArm.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 scale=0.001 0.001 0.001; visual mesh filename=package://bigman_urdf/meshes/walkman/BottomUpperArm.STL scale=0.001 0.001 0.001
- link RSoftHandLink: mass 1.2 -> 2.35; geometry collision mesh filename=package://bigman_urdf/meshes/walkman/simple/SoftHandOpen.STL scale=0.001 0.001 0.001; visual mesh filename=package://bigman_urdf/meshes/walkman/SoftHandOpen.STL scale=0.001 0.001 0.001
- link RThighLowLeg: mass 5.0950736 -> 5.31976; geometry collision mesh filename=package://bigman_urdf/meshes/walkman/simple/HipPitch.STL scale=0.001 0.001 0.001; visual mesh filename=package://bigman_urdf/meshes/walkman/HipPitch.STL scale=0.001 0.001 0.001
- link RThighUpLeg: mass 3.2402068 -> 3.06; geometry collision mesh filename=package://bigman_urdf/meshes/walkman/simple/HipYaw.STL scale=0.001 0.001 0.001; visual mesh filename=package://bigman_urdf/meshes/walkman/HipYaw.STL scale=0.001 0.001 0.001
- link RWrMot2: mass 1.2838072 -> 1.195; geometry collision mesh filename=package://bigman_urdf/meshes/walkman/simple/ForearmPitch.STL scale=0.001 0.001 0.001; visual mesh filename=package://bigman_urdf/meshes/walkman/ForearmPitch.STL scale=0.001 0.001 0.001
- link RWrMot3: mass 4.2801447e-01 -> 0.175; geometry collision mesh filename=package://bigman_urdf/meshes/walkman/simple/ForearmRoll.STL scale=0.001 0.001 0.001; visual mesh filename=package://bigman_urdf/meshes/walkman/ForearmRoll.STL scale=0.001 0.001 0.001
- link TorsoProtections: geometry collision mesh filename=package://bigman_urdf/meshes/walkman/simple/ProtectionSyste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 scale=0.001 0.001 0.001; visual mesh filename=package://bigman_urdf/meshes/walkman/ProtectionSystem.STL scale=0.001 0.001 0.001
- link Waist: mass 1.1046081e+01 -> 11.2; geometry collision mesh filename=package://bigman_urdf/meshes/walkman/simple/Waist.STL scale=0.001 0.001 0.001; visual mesh filename=package://bigman_urdf/meshes/walkman/Waist.STL scale=0.001 0.001 0.001
- link backpack: mass 10.0 -> 15.0
- link l_sole: mass 0 -> None
- link multisense/head: mass 1.41984 -> 4.105; geometry collision mesh filename=package://bigman_urdf/meshes/walkman/simple/Head.STL scale=0.001 0.001 0.001; visual mesh filename=package://bigman_urdf/meshes/walkman/Head.STL scale=0.001 0.001 0.001
- link multisense/hokuyo_link: mass 0.057654 -> 0.37; geometry collision box size=0.08 0.06 0.04238; collision cylinder length=0.047 radius=0.024425
- link r_sole: mass 0 -> None
Joints:
- added joint crane_ft_joint: type fixed, parent DWYTorso, child crane_ft, origin xyz=0 0 0.480 rpy=0 0 0
- joint LAnkLat: limit lower=-0.785 upper=0.785 effort=210 velocity=6.283 -> lower=-0.785 upper=0.785 effort=120 velocity=6.283
- joint LAnkSag: limit lower=-1.39556 upper=0.697778 effort=330 velocity=6.283 -> lower=-1.39556 upper=0.697778 effort=220 velocity=6.283
- joint LHipLat: limit lower=-0.697778 upper=0.87222 effort=400 velocity=6.283 -> lower=-0.697778 upper=0.87222 effort=220 velocity=6.283
- joint LHipSag: limit lower=-2.09333 upper=1.046667 effort=400 velocity=6.283 -> lower=-2.09333 upper=1.046667 effort=220 velocity=6.283
- joint LHipYaw: limit lower=-0.872222 upper=1.57 effort=140 velocity=6.283 -> lower=-0.872222 upper=1.57 effort=120 velocity=6.283
- joint LKneeSag: limit lower=0.0 upper=2.442222 effort=400 velocity=6.283 -> lower=0.0 upper=2.442222 effort=220 velocity=6.283
- joint LShSag: limit lower=-2.87979326578 upper=2.79252680318 effort=120 velocity=6.283 -> lower=-2.87979326578 upper=2.79252680318 effort=60 velocity=6.283
- joint NeckPitchj: origin xyz=0 0 0.117 rpy=0 0 0 -> xyz=0 0 0.1155 rpy=0 0 0
- joint RAnkLat: limit lower=-0.785 upper=0.785 effort=210 velocity=6.283 -> lower=-0.785 upper=0.785 effort=120 velocity=6.283
- joint RAnkSag: limit lower=-1.39556 upper=0.697778 effort=330 velocity=6.283 -> lower=-1.39556 upper=0.697778 effort=220 velocity=6.283
- joint RElbj: limit lower=-2.96705972838 upper=0.593411945677 effort=120 velocity=6.283 -> lower=-2.96705972838 upper=0.593411945677 effort=60 velocity=6.283
- joint RHipLat: limit lower=-0.87222 upper=0.697778 effort=400 velocity=6.283 -> lower=-0.87222 upper=0.697778 effort=220 velocity=6.283
- joint RHipSag: limit lower=-2.09333 upper=1.046667 effort=400 velocity=6.283 -> lower=-2.09333 upper=1.046667 effort=220 velocity=6.283
- joint RHipYaw: limit lower=-1.57 upper=0.872222 effort=140 velocity=6.283 -> lower=-1.57 upper=0.872222 effort=120 velocity=6.283
- joint RKneeSag: limit lower=0.0 upper=2.442222 effort=400 velocity=6.283 -> lower=0.0 upper=2.442222 effort=220 velocity=6.283
