Commit message: adding contacts on the legs in iCubGenova04 model

File: app/robots/iCubGenova04/model.urdf (robot description, URDF)
Before this commit: robot ICUB_2-5_BB_SIM_MODEL, 163 links, 162 joints
Links:
- added link l_upper_leg_contact
- added link r_upper_leg_contact
Joints:
- added joint l_upper_leg_contact_fixed_joint: type fixed, parent l_upper_leg, child l_upper_leg_contact, origin xyz=-0.0003 0.0146 -0.0512571 rpy=0 0 -1.57079632679
- added joint r_upper_leg_contact_fixed_joint: type fixed, parent r_upper_leg, child r_upper_leg_contact, origin xyz=0.0003 0.0146 -0.0512571 rpy=0 0 -1.57079632679
